File: PCB/Poor86.kicad_pcb (KiCad board)
At the start: 4 copper layers, 100 x 170 mm, 101 parts, among them J1 Bus_ISA_8bit, J3 ATX-20, P1 USB_C_Plug_USB2.0, SW3 SW_Push_Dual, SW4 SW_Push_Dual, U1 LFE5U-25F-6BG256C, U11 CH552T, U12 IS66WVH8M8BLL-100B1LI, U13 IS66WVH8M8BLL-100B1LI, U14 KM416x254, U15 KM416x254, U2 TLV62569DBV, U3 AM5x86 PQFP208, U4 TLV62569DBV, U5 ESP-12F, U6 TLV62569DBV, U7 RP2354B, U8 CL-GD5428-LOCALBUS

Commit message: started initial layout
Parts:
- added U16: SN74ALVC164245DGG, Package_SO:TSSOP-48_6.1x12.5mm_P0.5mm, F.Cu at (-59.8, 25.5)
- added U17: SN74ALVC164245DGG, Package_SO:TSSOP-48_6.1x12.5mm_P0.5mm, F.Cu at (-73.0, 25.5)
- moved J3 145.8 mm to (169.5, -75.0)
- moved SW3 145.8 mm to (175.0, -54.5)
- moved SW4 145.8 mm to (175.0, -63.0)
- moved U14 129.9 mm to (-49.4, -11.8)
- moved C9 120.0 mm to (57.1, 21.4), turned to -90 degrees
- moved C6 115.5 mm to (68.1, 21.4), turned to -90 degrees
- moved C8 115.2 mm to (69.6, 21.4), turned to -90 degrees
- moved CDC1 111.0 mm to (132.8, 28.9)
- moved CDC10 111.0 mm to (135.7, 27.0)
- moved CDC11 111.0 mm to (135.7, 25.0)
- moved CDC12 111.0 mm to (135.7, 23.0)
- moved CDC13 111.0 mm to (135.7, 21.1)
- moved CDC14 111.0 mm to (135.7, 19.1)
- moved CDC15 111.0 mm to (135.7, 17.1)
- moved CDC16 111.0 mm to (135.7, 15.2)
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Connections:
- net /VideoSubSystem/2/1xCLK renamed /VideoSubSystem/CLK_CPU
- net /VideoSubSystem/A1/~{BE3} renamed /VideoSubSystem/~{BE3}
- net /VideoSubSystem/M/~{IO} renamed /VideoSubSystem/M~{IO}
- net /VideoSubSystem/NC/~{BE0} renamed /VideoSubSystem/~{BE0}
- net /VideoSubSystem/NC/~{BS16}/~{LDS16} renamed /VideoSubSystem/~{BS16}
- net /VideoSubSystem/NC/~{UADDR} renamed /VideoSubSystem/~{UADDR_VGA}
- net /VideoSubSystem/W/~{R} renamed /VideoSubSystem/W~{R}
- net /VideoSubSystem/~{ADS} renamed /VideoSubSystem/~{RDY_CPU}
- net /VideoSubSystem/~{BHE}/~{BE1} renamed /VideoSubSystem/~{BE1}
- net /VideoSubSystem/~{BLE}/~{BE2} renamed /VideoSubSystem/~{BE2}
- net /VideoSubSystem/~{LBA} renamed /VideoSubSystem/~{LBA_VGA}
- net /VideoSubSystem/~{READY} renamed /VideoSubSystem/~{ADS_CPU}
- net /am5x86/A24 renamed A24
- net /am5x86/A25 renamed A25
- net /am5x86/A26 renamed A26
- net /am5x86/A27 renamed A27
- net /am5x86/A28 renamed A28
- net /am5x86/A29 renamed A29
- net /am5x86/A30 renamed A30
- net /am5x86/A31 renamed A31
- U14 pad 13: unconnected-(U14-~{W}-Pad13) -> /VideoSubSystem/CAS
- U14 pad 14: unconnected-(U14-~{RAS}-Pad14) -> /VideoSubSystem/OE
- U14 pad 27: unconnected-(U14-~{OE}-Pad27) -> GNDD
- U14 pad 28: Net-(U14-~{LCAS}) -> /VideoSubSystem/WE3
- U14 pad 29: Net-(U14-~{LCAS}) -> /VideoSubSystem/WE2
- U15 pad 13: unconnected-(U15-~{W}-Pad13) -> /VideoSubSystem/CAS
- U15 pad 14: unconnected-(U15-~{RAS}-Pad14) -> /VideoSubSystem/RAS
- U15 pad 27: unconnected-(U15-~{OE}-Pad27) -> GNDD
- U15 pad 28: unconnected-(U15-~{UCAS}-Pad28) -> /VideoSubSystem/WE1
- U15 pad 29: unconnected-(U15-~{LCAS}-Pad29) -> /VideoSubSystem/WE0
- U3 pad 11: unconnected-(U3B-CLKMUL-Pad11) -> /am5x86/CLKMUL
- U3 pad 12: unconnected-(U3B-~{RDY}-Pad12) -> /am5x86/~{RDY_CPU}
- U3 pad 159: /am5x86/A23 -> A23
- U3 pad 160: /am5x86/A22 -> A22
- U3 pad 161: /am5x86/A21 -> A21
- U3 pad 164: /am5x86/A20 -> A20
- U3 pad 165: /am5x86/A19 -> A19
- U3 pad 166: /am5x86/A18 -> A18
- U3 pad 171: /am5x86/A17 -> A17
- U3 pad 173: /am5x86/A16 -> A16
- U3 pad 174: /am5x86/A15 -> A15
- U3 pad 177: /am5x86/A14 -> A14
- U3 pad 178: /am5x86/A13 -> A13
- U3 pad 180: /am5x86/A12 -> A12
- U3 pad 182: /am5x86/A11 -> A11
- U3 pad 186: /am5x86/A10 -> A10
- U3 pad 187: /am5x86/A9 -> A9
- U3 pad 190: /am5x86/A8 -> A8
- U3 pad 192: /am5x86/A7 -> A7
- U3 pad 193: /am5x86/A6 -> A6
- U3 pad 195: /am5x86/A5 -> A5
- U3 pad 196: /am5x86/A4 -> A4
- U3 pad 197: /am5x86/A3 -> A3
- U3 pad 202: /am5x86/A2 -> A2
- U3 pad 203: unconnected-(U3B-~{ADS}-Pad203) -> /am5x86/~{ADS_CPU}
- U3 pad 206: unconnected-(U3B-~{PLOCK}-Pad206) -> /am5x86/~{PLOCK}
- U3 pad 207: unconnected-(U3B-~{LOCK}-Pad207) -> /am5x86/~{LOCK}
- U3 pad 24: unconnected-(U3B-CLK-Pad24) -> /am5x86/CLK_CPU
- U3 pad 27: unconnected-(U3B-W~{R}-Pad27) -> /am5x86/W~{R}
- U3 pad 31: unconnected-(U3B-~{BE0}-Pad31) -> /am5x86/~{BE0}
- U3 pad 32: unconnected-(U3B-~{BE1}-Pad32) -> /am5x86/~{BE1}
- U3 pad 33: unconnected-(U3B-~{BE2}-Pad33) -> /am5x86/~{BE2}
- U3 pad 34: unconnected-(U3B-~{BE3}-Pad34) -> /am5x86/~{BE3}
- U3 pad 37: unconnected-(U3B-M~{IO}-Pad37) -> /am5x86/M~{IO}
- U3 pad 39: unconnected-(U3B-D~{C}-Pad39) -> /am5x86/D~{C}
- U3 pad 47: unconnected-(U3B-~{A20M}-Pad47) -> /am5x86/~{A20M}
- U3 pad 7: unconnected-(U3B-~{BS16}-Pad7) -> /am5x86/~{BS16}
- U3 pad 73: unconnected-(U3B-~{STPCLK}-Pad73) -> /am5x86/~{STPCLK}
- U3 pad 8: unconnected-(U3B-~{BS8}-Pad8) -> /am5x86/~{BS8}
- U8 pad 15: /VideoSubSystem/A17 -> A17
- U8 pad 16: /VideoSubSystem/A18 -> A18
- U8 pad 17: /VideoSubSystem/A19 -> A19
- U8 pad 18: /VideoSubSystem/A20 -> A20
- U8 pad 19: /VideoSubSystem/A21 -> A21
- U8 pad 20: /VideoSubSystem/A22 -> A22
- U8 pad 21: /VideoSubSystem/A23 -> A23
- U8 pad 29: /VideoSubSystem/A2 -> A2
- U8 pad 30: /VideoSubSystem/A3 -> A3
- U8 pad 31: /VideoSubSystem/A4 -> A4
- U8 pad 32: /VideoSubSystem/A5 -> A5
- U8 pad 33: /VideoSubSystem/A6 -> A6
- U8 pad 34: /VideoSubSystem/A7 -> A7
- U8 pad 35: /VideoSubSystem/A8 -> A8
- U8 pad 36: /VideoSubSystem/A9 -> A9
- U8 pad 37: /VideoSubSystem/A10 -> A10
- U8 pad 38: /VideoSubSystem/A11 -> A11
- U8 pad 39: /VideoSubSystem/A12 -> A12
- U8 pad 41: /VideoSubSystem/RESET -> unconnected-(U8-RESET-Pad41)
- U8 pad 42: /VideoSubSystem/A13 -> A13
- U8 pad 43: /VideoSubSystem/A14 -> A14
- U8 pad 44: /VideoSubSystem/A15 -> A15
- U8 pad 45: /VideoSubSystem/A16 -> A16
- U8 pad 46: /VideoSubSystem/CPU_RESET -> unconnected-(U8-CPU_RESET-Pad46)
- U8 pad 51: (no net) -> GNDD
- U8 pad 52: /VideoSubSystem/INTR -> unconnected-(U8-INTR-Pad52)
- U8 pad 73: /VideoSubSystem/EEDI -> /VideoSubSystem/~{OE_H}
- U8 pad 74: /VideoSubSystem/EECS -> /VideoSubSystem/~{OE_L}
Routing:
- net A2: track 0.00 -> 68.2 mm
- net A3: track 0.00 -> 66.4 mm
- net A4: track 0.00 -> 65.5 mm
- net A5: track 0.00 -> 64.5 mm
- net A6: track 0.00 -> 63.4 mm
- net A7: track 0.00 -> 62.4 mm
- net A8: track 0.00 -> 61.3 mm
- net A9: track 0.00 -> 59.9 mm
- net A10: track 0.00 -> 59.0 mm
- net A11: track 0.00 -> 55.5 mm
- net A12: track 0.00 -> 54.2 mm
- net A13: track 0.00 -> 51.5 mm
- net A14: track 0.00 -> 51.3 mm
- net A15: track 0.00 -> 50.6 mm
- net A16: track 0.00 -> 50.4 mm
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Other:
- board text added: "Address"
- board text added: "BUS"
- board text added: "Command"
- board text added: "Data"
- board text added: "MEM"
- board text added: "VID"

Commit message: More layout work
Parts:
- removed C1, C16, C25: 100pF, Capacitor_SMD:C_0402_1005Metric
- removed C10, C14, C23, C32, C33, C5, C6, C7, C8, C9: 47uF, Capacitor_SMD:C_0603_1608Metric
- removed C11, C12, C13, C17, C18, C19, C2, C20, C21, C22, C26, C27, C28, C29, C3, C30, C31, C4: 1u, Capacitor_SMD:C_0402_1005Metric
- removed C15, C24: 10uF, Capacitor_SMD:C_0603_1608Metric
- removed CDC1, CDC10, CDC11, CDC12, CDC13, CDC14, CDC15, CDC16, CDC17, CDC18, CDC19, CDC2, CDC20, CDC21, CDC22, CDC23, CDC24, CDC25, CDC26, CDC27, CDC28, CDC29, CDC3, CDC30, CDC31, CDC32, CDC33, CDC34, CDC35, CDC36, CDC37, CDC38, CDC4, CDC5, CDC6, CDC7, CDC8, CDC9: 1uF, Capacitor_SMD:C_0402_1005Metric
- removed JP1: Closed=3.3V, Open=3.5V, Jumper:SolderJumper-2_P1.3mm_Bridged_Pad1.0x1.5mm
- removed L1, L2, L3: 2.2uH, Inductor_SMD:L_1008_2520Metric
- removed R1, R3, R5: 15k, Resistor_SMD:R_0402_1005Metric
- removed R2: 18k, Resistor_SMD:R_0402_1005Metric
- removed R4: 4.7K, Resistor_SMD:R_0402_1005Metric
- removed R6: 3.3k, Resistor_SMD:R_0402_1005Metric
- removed R7: 1k, Resistor_SMD:R_0402_1005Metric
- moved U4 173.7 mm to (2.08, 6.53), turned to 0 degrees
- moved U15 170.2 mm to (75.2, 117.3), turned to 180 degrees
- moved U14 167.2 mm to (57.0, 117.3), turned to 180 degrees
- moved U2 161.8 mm to (2.08, 1.90), turned to 0 degrees
- moved U6 140.5 mm to (2.08, 11.2), turned to 0 degrees
- moved U16 131.4 mm to (66.3, 62.7), turned to -90 degrees
- moved U17 129.6 mm to (51.1, 62.7), turned to -90 degrees
- moved U12 78.6 mm to (-12.0, 22.8)
- moved U13 78.6 mm to (-12.0, 14.8)
- moved U1 57.7 mm to (30.1, 59.7)
Connections:
- net /am5x86/CLKMUL renamed CLKMUL
- net /am5x86/D~{C} renamed D~{C}
- net /am5x86/~{A20M} renamed ~{A20M}
- net /am5x86/~{BS8} renamed ~{BS8}
- net /am5x86/~{LOCK} renamed ~{LOCK}
- net /am5x86/~{PLOCK} renamed ~{PLOCK}
- net /am5x86/~{STPCLK} renamed ~{STPCLK}
- U16 pad 1: unconnected-(U16-1DIR-Pad1) -> W~{R}
- U16 pad 10: Net-(U16-GND-Pad10) -> GNDD
- U16 pad 11: unconnected-(U16-1B6-Pad11) -> D6
- U16 pad 12: unconnected-(U16-1B7-Pad12) -> D7
- U16 pad 13: unconnected-(U16-2B0-Pad13) -> D8
- U16 pad 14: unconnected-(U16-2B1-Pad14) -> D9
- U16 pad 15: Net-(U16-GND-Pad10) -> GNDD
- U16 pad 16: unconnected-(U16-2B2-Pad16) -> D10
- U16 pad 17: unconnected-(U16-2B3-Pad17) -> D11
- U16 pad 19: unconnected-(U16-2B4-Pad19) -> D12
- U16 pad 2: unconnected-(U16-1B0-Pad2) -> D0
- U16 pad 20: unconnected-(U16-2B5-Pad20) -> D13
- U16 pad 21: Net-(U16-GND-Pad10) -> GNDD
- U16 pad 22: unconnected-(U16-2B6-Pad22) -> D14
- U16 pad 23: unconnected-(U16-2B7-Pad23) -> D15
- U16 pad 24: unconnected-(U16-2DIR-Pad24) -> W~{R}
- U16 pad 28: Net-(U16-GND-Pad10) -> GNDD
- U16 pad 3: unconnected-(U16-1B1-Pad3) -> D1
- U16 pad 31: Net-(U16-V_{CC(A)}-Pad31) -> +5V
- U16 pad 34: Net-(U16-GND-Pad10) -> GNDD
- U16 pad 39: Net-(U16-GND-Pad10) -> GNDD
- U16 pad 4: Net-(U16-GND-Pad10) -> GNDD
- U16 pad 42: Net-(U16-V_{CC(A)}-Pad31) -> +5V
- U16 pad 45: Net-(U16-GND-Pad10) -> GNDD
- U16 pad 5: unconnected-(U16-1B2-Pad5) -> D2
- U16 pad 6: unconnected-(U16-1B3-Pad6) -> D3
- U16 pad 8: unconnected-(U16-1B4-Pad8) -> D4
- U16 pad 9: unconnected-(U16-1B5-Pad9) -> D5
- U17 pad 1: unconnected-(U17-1DIR-Pad1) -> W~{R}
- U17 pad 10: Net-(U17-GND-Pad10) -> GNDD
- U17 pad 11: unconnected-(U17-1B6-Pad11) -> D22
- U17 pad 12: unconnected-(U17-1B7-Pad12) -> D23
- U17 pad 13: unconnected-(U17-2B0-Pad13) -> D24
- U17 pad 14: unconnected-(U17-2B1-Pad14) -> D25
- U17 pad 15: Net-(U17-GND-Pad10) -> GNDD
- U17 pad 16: unconnected-(U17-2B2-Pad16) -> D26
- U17 pad 17: unconnected-(U17-2B3-Pad17) -> D27
- U17 pad 19: unconnected-(U17-2B4-Pad19) -> D28
- U17 pad 2: unconnected-(U17-1B0-Pad2) -> D16
- U17 pad 20: unconnected-(U17-2B5-Pad20) -> D29
- U17 pad 21: Net-(U17-GND-Pad10) -> GNDD
- U17 pad 22: unconnected-(U17-2B6-Pad22) -> D30
- U17 pad 23: unconnected-(U17-2B7-Pad23) -> D31
- U17 pad 24: unconnected-(U17-2DIR-Pad24) -> W~{R}
- U17 pad 28: Net-(U17-GND-Pad10) -> GNDD
- U17 pad 3: unconnected-(U17-1B1-Pad3) -> D17
- U17 pad 31: Net-(U17-V_{CC(A)}-Pad31) -> +5V
- U17 pad 34: Net-(U17-GND-Pad10) -> GNDD
- U17 pad 39: Net-(U17-GND-Pad10) -> GNDD
- U17 pad 4: Net-(U17-GND-Pad10) -> GNDD
- U17 pad 42: Net-(U17-V_{CC(A)}-Pad31) -> +5V
- U17 pad 45: Net-(U17-GND-Pad10) -> GNDD
- U17 pad 5: unconnected-(U17-1B2-Pad5) -> D18
- U17 pad 6: unconnected-(U17-1B3-Pad6) -> D19
- U17 pad 8: unconnected-(U17-1B4-Pad8) -> D20
- U17 pad 9: unconnected-(U17-1B5-Pad9) -> D21
- U3 pad 100: /am5x86/D19 -> D19
- U3 pad 101: /am5x86/D18 -> D18
- U3 pad 103: /am5x86/D17 -> D17
- U3 pad 108: /am5x86/D16 -> D16
- U3 pad 112: /am5x86/D15 -> D15
- U3 pad 113: /am5x86/D14 -> D14
- U3 pad 116: /am5x86/D13 -> D13
- U3 pad 117: /am5x86/D12 -> D12
- U3 pad 118: /am5x86/D11 -> D11
- U3 pad 119: /am5x86/D10 -> D10
- U3 pad 12: /am5x86/~{RDY_CPU} -> ~{RDY}
- U3 pad 123: /am5x86/D9 -> D9
- U3 pad 124: /am5x86/D8 -> D8
- U3 pad 126: /am5x86/D7 -> D7
- U3 pad 129: /am5x86/D6 -> D6
- U3 pad 130: /am5x86/D5 -> D5
- U3 pad 140: /am5x86/D4 -> D4
- U3 pad 141: /am5x86/D3 -> D3
- U3 pad 142: /am5x86/D2 -> D2
- U3 pad 143: /am5x86/D1 -> D1
- U3 pad 144: /am5x86/D0 -> D0
- U3 pad 194: unconnected-(U3B-~{UP}-Pad194) -> ~{UP}
- U3 pad 203: /am5x86/~{ADS_CPU} -> ~{ADS}
- U3 pad 24: /am5x86/CLK_CPU -> CLK
- U3 pad 27: /am5x86/W~{R} -> W~{R}
- U3 pad 31: /am5x86/~{BE0} -> ~{BE0}
- U3 pad 32: /am5x86/~{BE1} -> ~{BE1}
- U3 pad 33: /am5x86/~{BE2} -> ~{BE2}
- U3 pad 34: /am5x86/~{BE3} -> ~{BE3}
- U3 pad 37: /am5x86/M~{IO} -> M~{IO}
- U3 pad 48: unconnected-(U3B-RESET-Pad48) -> RESET
- U3 pad 50: unconnected-(U3B-INTR-Pad50) -> INTR
- U3 pad 51: unconnected-(U3B-NMI-Pad51) -> NMI
- U3 pad 58: unconnected-(U3B-SRESET-Pad58) -> SRESET
- U3 pad 7: /am5x86/~{BS16} -> ~{BS16}
- U3 pad 74: /am5x86/D31 -> D31
- U3 pad 75: /am5x86/D30 -> D30
- U3 pad 78: /am5x86/D29 -> D29
- U3 pad 79: /am5x86/D28 -> D28
- U3 pad 83: /am5x86/D27 -> D27
- U3 pad 84: /am5x86/D26 -> D26
- U3 pad 85: /am5x86/D25 -> D25
- U3 pad 87: /am5x86/D24 -> D24
- U3 pad 91: /am5x86/D23 -> D23
- U3 pad 92: /am5x86/D22 -> D22
- U3 pad 93: /am5x86/D21 -> D21
- U3 pad 99: /am5x86/D20 -> D20
- U8 pad 10: /VideoSubSystem/D9 -> /VideoSubSystem/2A1
- U8 pad 11: /VideoSubSystem/D8 -> /VideoSubSystem/2A0
- U8 pad 13: /VideoSubSystem/~{UADDR_VGA} -> unconnected-(U8-NC/~{UADDR}-Pad13)
- U8 pad 14: /VideoSubSystem/M~{IO} -> M~{IO}
- U8 pad 22: /VideoSubSystem/~{LBA_VGA} -> unconnected-(U8-~{LBA}-Pad22)
- U8 pad 23: /VideoSubSystem/~{BS16} -> ~{BS16}
- U8 pad 24: /VideoSubSystem/~{BE1} -> ~{BE1}
- U8 pad 25: /VideoSubSystem/~{RDY_CPU} -> ~{ADS}
- U8 pad 27: /VideoSubSystem/~{BE2} -> ~{BE2}
- U8 pad 28: /VideoSubSystem/~{BE3} -> ~{BE3}
- U8 pad 3: /VideoSubSystem/D15 -> /VideoSubSystem/2A7
- U8 pad 4: /VideoSubSystem/D14 -> /VideoSubSystem/2A6
- U8 pad 46: unconnected-(U8-CPU_RESET-Pad46) -> RESET
- U8 pad 47: /VideoSubSystem/~{ADS_CPU} -> ~{RDY}
- U8 pad 48: /VideoSubSystem/~{BE0} -> ~{BE0}
- U8 pad 49: /VideoSubSystem/W~{R} -> W~{R}
- U8 pad 5: /VideoSubSystem/D13 -> /VideoSubSystem/2A5
- U8 pad 50: /VideoSubSystem/CLK_CPU -> CLK
- U8 pad 54: /VideoSubSystem/D0 -> /VideoSubSystem/1A0
- U8 pad 55: /VideoSubSystem/D1 -> /VideoSubSystem/1A1
- U8 pad 56: /VideoSubSystem/D2 -> /VideoSubSystem/1A2
- U8 pad 57: /VideoSubSystem/D3 -> /VideoSubSystem/1A3
- U8 pad 59: /VideoSubSystem/D4 -> /VideoSubSystem/1A4
- U8 pad 6: /VideoSubSystem/D12 -> /VideoSubSystem/2A4
- U8 pad 60: /VideoSubSystem/D5 -> /VideoSubSystem/1A5
- U8 pad 62: /VideoSubSystem/D6 -> /VideoSubSystem/1A6
- U8 pad 63: /VideoSubSystem/D7 -> /VideoSubSystem/1A7
- U8 pad 8: /VideoSubSystem/D11 -> /VideoSubSystem/2A3
- U8 pad 9: /VideoSubSystem/D10 -> /VideoSubSystem/2A2
Routing:
- net /VideoSubSystem/2A7: track 0.00 -> 73.6 mm, vias 0 -> 3
- net /VideoSubSystem/2A6: track 0.00 -> 71.9 mm, vias 0 -> 3
- net /VideoSubSystem/2A5: track 0.00 -> 70.6 mm, vias 0 -> 3
- net /VideoSubSystem/2A4: track 0.00 -> 69.1 mm, vias 0 -> 3
- net /VideoSubSystem/2A3: track 0.00 -> 66.9 mm, vias 0 -> 3
- net /VideoSubSystem/2A2: track 0.00 -> 65.3 mm, vias 0 -> 3
- net /VideoSubSystem/2A1: track 0.00 -> 63.8 mm, vias 0 -> 3
- net /VideoSubSystem/2A0: track 0.00 -> 62.3 mm, vias 0 -> 3
- net A17: track 9.01 -> 63.9 mm, vias 0 -> 3
- net W~{R}: track 0.00 -> 46.7 mm, vias 0 -> 4
- net A18: track 14.3 -> 60.8 mm, vias 0 -> 2
- net A19: track 12.7 -> 59.1 mm, vias 0 -> 2
- net A20: track 13.6 -> 57.7 mm, vias 0 -> 2
- net A21: track 25.2 -> 55.4 mm, vias 0 -> 2
- net A23: track 23.1 -> 52.7 mm, vias 1 -> 2
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