File: PCB/Poor86.kicad_pcb (KiCad board)
At the start: 4 copper layers, 100 x 170 mm, 21 parts, among them J1 Bus_ISA_8bit, J3 ATX-20, P1 USB_C_Plug_USB2.0, SW3 SW_Push_Dual, SW4 SW_Push_Dual, U1 LFE5U-25F-6BG256C, U11 CH552T, U12 IS66WVH8M8BLL-100B1LI, U13 IS66WVH8M8BLL-100B1LI, U14 KM416x254, U15 KM416x254, U16 SN74ALVC164245DGG, U17 SN74ALVC164245DGG, U2 TLV62569DBV, U3 AM5x86 PQFP208, U4 TLV62569DBV, U5 ESP-12F, U6 TLV62569DBV, U7 RP2354B, U8 CL-GD5428-LOCALBUS

Commit message: route-out in progress
Parts:
- removed J1: Bus_ISA_8bit, ISA:TE_7-5530843-0
- removed J3: ATX-20, Connector_Molex:Molex_Mini-Fit_Jr_5566-20A_2x10_P4.20mm_Vertical
- removed U13: IS66WVH8M8BLL-100B1LI, Package_BGA:BGA-24_6x8mm_Layout5x5_P1.0mm
- removed U14, U15: KM416x254, Package_SO:TSOP-II-40-44_10.16x18.37mm_P0.8mm
- removed U16, U17: SN74ALVC164245DGG, Package_SO:TSSOP-48_6.1x12.5mm_P0.5mm
- removed U7: RP2354B, Package_DFN_QFN:QFN-80-1EP_10x10mm_P0.4mm_EP3.4x3.4mm
- removed U8: CL-GD5428-LOCALBUS, Package_QFP:PQFP-160_28x28mm_P0.65mm
- added C35: 2.2nF, Capacitor_SMD:C_01005_0402Metric, F.Cu at (22.4, 66.9)
- added C36: 2.2nF, Capacitor_SMD:C_01005_0402Metric, F.Cu at (22.4, 66.1)
- added C45: 2.2nF, Capacitor_SMD:C_01005_0402Metric, F.Cu at (22.4, 65.2)
- added C46: 2.2nF, Capacitor_SMD:C_01005_0402Metric, F.Cu at (22.4, 64.6)
- added C47: 2.2nF, Capacitor_SMD:C_01005_0402Metric, F.Cu at (22.4, 63.9)
- added C48: 2.2nF, Capacitor_SMD:C_01005_0402Metric, F.Cu at (22.4, 63.3)
- added C49: 2.2nF, Capacitor_SMD:C_01005_0402Metric, F.Cu at (22.4, 62.7)
- added C50: 2.2nF, Capacitor_SMD:C_01005_0402Metric, F.Cu at (22.4, 62.1)
- added J5: 10018783-10202TLF, 10018783_10202TLF:AMPHENOL_10018783-10202TLF, F.Cu at (29.6, 76.8)
- added J6: HDMI_A, Connector_Video:HDMI_A_Amphenol_10029449-x01xLF_Horizontal, F.Cu at (15.2, 62.6)
- added U18: 4068, Package_SO:TSSOP-14_4.4x5mm_P0.65mm, F.Cu at (43.0, 51.8)
- added Y1: CMOS-50MHz, Oscillator:Oscillator_SMD_Abracon_ASE-4Pin_3.2x2.5mm, F.Cu at (25.0, 70.4)
- U5: moved to B.Cu
- moved SW3 139.6 mm to (53.8, 14.8), turned to 0 degrees
- moved SW4 135.7 mm to (63.8, 14.8), turned to 0 degrees
- moved P1 119.4 mm to (68.0, 27.0), turned to 90 degrees
- moved U11 113.0 mm to (58.9, 26.9), turned to 0 degrees
- moved D1 105.3 mm to (70.4, 47.3), turned to 90 degrees
- moved U5 93.2 mm to (67.6, 41.7)
- moved U2 77.5 mm to (66.3, 45.3), turned to 180 degrees
- moved U4 72.7 mm to (66.3, 40.6), turned to 180 degrees
- moved U6 68.8 mm to (66.3, 36.0), turned to 180 degrees
- moved U12 67.2 mm to (44.0, 59.9), turned to 0 degrees
- moved U3 35.0 mm to (31.9, 31.5)
- moved U1 1.28 mm to (31.0, 60.6), turned to 0 degrees
Connections:
- net CLKMUL renamed Net-(JP3-B)
- net ~{UP} renamed Net-(JP2-B)
- U1 pad A10: unconnected-(U1B-PT42B-PadA10) -> ~{A20M}
- U1 pad A11: unconnected-(U1B-PT53A-PadA11) -> PCD
- U1 pad A12: unconnected-(U1B-PT53B-PadA12) -> PWT
- U1 pad A13: unconnected-(U1B-PT65A-PadA13) -> D~{C}
- U1 pad A14: unconnected-(U1B-PT65B-PadA14) -> D7
- U1 pad A15: unconnected-(U1B-PT67B-PadA15) -> ~{BE2}
- U1 pad A2: unconnected-(U1A-PT4A-PadA2) -> ~{CACHE}
- U1 pad A3: unconnected-(U1A-PT6A-PadA3) -> D15
- U1 pad A4: unconnected-(U1A-PT6B-PadA4) -> D14
- U1 pad A5: unconnected-(U1A-PT18A-PadA5) -> ~{SMIACT}
- U1 pad A6: unconnected-(U1A-PT18B-PadA6) -> D13
- U1 pad A7: unconnected-(U1A-PT29A-PadA7) -> D12
- U1 pad A8: unconnected-(U1A-PT29B-PadA8) -> D11
- U1 pad A9: unconnected-(U1B-PT42A-PadA9) -> D10
- U1 pad B1: unconnected-(U1F-PL2A-PadB1) -> D16
- U1 pad B10: unconnected-(U1B-PT44A-PadB10) -> RESET
- U1 pad B11: unconnected-(U1B-PT49A-PadB11) -> ~{EADS}
- U1 pad B12: unconnected-(U1B-PT56A-PadB12) -> D9
- U1 pad B13: unconnected-(U1B-PT60A-PadB13) -> D8
- U1 pad B14: unconnected-(U1B-PT67A-PadB14) -> M~{IO}
- U1 pad B15: unconnected-(U1C-PR2B-PadB15) -> ~{BE3}
- U1 pad B16: unconnected-(U1C-PR2A-PadB16) -> ~{BE1}
- U1 pad B2: unconnected-(U1F-PL2B-PadB2) -> INV
- U1 pad B3: unconnected-(U1A-PT4B-PadB3) -> ~{SMI}
- U1 pad B4: unconnected-(U1A-PT11B-PadB4) -> WB~{WT}
- U1 pad B5: unconnected-(U1A-PT15B-PadB5) -> ~{HITM}
- U1 pad B6: unconnected-(U1A-PT22B-PadB6) -> SRESET
- U1 pad B7: unconnected-(U1A-PT27B-PadB7) -> NMI
- U1 pad B8: unconnected-(U1B-PT35B-PadB8) -> INTR
- U1 pad B9: unconnected-(U1B-PT38A-PadB9) -> ~{FLUSH}
- U1 pad C1: unconnected-(U1F-PL5A-PadC1) -> D18
- U1 pad C14: unconnected-(U1C-PR2C-PadC14) -> W~{R}
- U1 pad C15: unconnected-(U1C-PR5B-PadC15) -> ~{BE0}
- U1 pad C16: unconnected-(U1C-PR5A-PadC16) -> BREQ
- U1 pad C2: unconnected-(U1F-PL5B-PadC2) -> D17
- U1 pad C9: unconnected-(U1B-PT38B-PadC9) -> D5
- U1 pad D16: unconnected-(U1C-PR8A-PadD16) -> HOLDA
- U1 pad D9: unconnected-(U1B-PT40A-PadD9) -> D6
- U1 pad E15: unconnected-(U1C-PR8B-PadE15) -> CLK
- U1 pad E16: unconnected-(U1C-PR11D-PadE16) -> UADDR
- U1 pad F10: VCCIO1 -> +3V3
- U1 pad F11: VCCIO1 -> +3V3
- U1 pad F15: unconnected-(U1C-PR11C-PadF15) -> A25
- U1 pad F16: unconnected-(U1C-PR14A-PadF16) -> /Memory/OB_CLKt
- U1 pad F6: VCCIO0 -> +3V3
- U1 pad F7: VCCIO0 -> +3V3
- U1 pad G14: unconnected-(U1C-PR14C-PadG14) -> /Memory/~{RESET}
- U1 pad G15: unconnected-(U1C-PR14B-PadG15) -> /Memory/~{CS}
- U1 pad G16: unconnected-(U1C-PR20A-PadG16) -> /Memory/OB_RWDS
- U1 pad H11: VCCIO2 -> +3V3
- U1 pad H15: unconnected-(U1C-PR20B-PadH15) -> /Memory/DQ2
- U1 pad H6: VCCIO7 -> +3V3
- U1 pad H7: VCCIO7 -> +3V3
- U1 pad J11: VCCIO2 -> +3V3
- U1 pad J13: unconnected-(U1C-PR17C-PadJ13) -> /Memory/DQ5
- U1 pad J14: unconnected-(U1C-PR20C-PadJ14) -> /Memory/DQ1
- U1 pad J15: unconnected-(U1C-PR23B-PadJ15) -> /Memory/DQ0
- U1 pad J16: unconnected-(U1C-PR23A-PadJ16) -> /Memory/DQ4
- U1 pad J6: VCCIO6 -> +3V3
- U1 pad J7: VCCIO6 -> +3V3
- U1 pad K11: VCCIO3 -> +3V3
- U1 pad K14: unconnected-(U1C-PR20D-PadK14) -> /Memory/DQ6
- U1 pad K15: unconnected-(U1C-PR23D-PadK15) -> /Memory/DQ7
- U1 pad K16: unconnected-(U1C-PR23C-PadK16) -> /Memory/DQ3
- U1 pad L1: unconnected-(U1E-PL26A-PadL1) -> /eternal_perif/CK+
- U1 pad L11: VCCIO3 -> +3V3
- U1 pad L15: unconnected-(U1D-PR26B-PadL15) -> A23
- U1 pad L16: unconnected-(U1D-PR26A-PadL16) -> A24
- U1 pad L2: unconnected-(U1E-PL26B-PadL2) -> /eternal_perif/CK-
- U1 pad L6: unconnected-(U1G-VCCIO8-PadL6) -> +3V3
- U1 pad M1: unconnected-(U1E-PL26C-PadM1) -> /eternal_perif/D0+
- U1 pad M15: unconnected-(U1D-PR26D-PadM15) -> A21
- U1 pad M16: unconnected-(U1D-PR26C-PadM16) -> A22
- U1 pad M2: unconnected-(U1E-PL26D-PadM2) -> /eternal_perif/D0-
- U1 pad N1: unconnected-(U1E-PL32A-PadN1) -> /eternal_perif/D1+
- U1 pad N14: unconnected-(U1D-PR35D-PadN14) -> A19
- U1 pad N16: unconnected-(U1D-PR32A-PadN16) -> A20
- U1 pad P1: unconnected-(U1E-PL35A-PadP1) -> /eternal_perif/D2+
- U1 pad P11: unconnected-(U1D-PR47C-PadP11) -> LRC_GPLL0T_IN
- U1 pad P15: unconnected-(U1D-PR32B-PadP15) -> A17
- U1 pad P16: unconnected-(U1D-PR35A-PadP16) -> A18
- U1 pad P2: unconnected-(U1E-PL32B-PadP2) -> /eternal_perif/D1-
- U1 pad R1: unconnected-(U1E-PL35B-PadR1) -> /eternal_perif/D2-
- U1 pad R10: unconnected-(U1G-CFG_2-PadR10) -> A8
- U1 pad R12: unconnected-(U1D-PR44A-PadR12) -> A9
- U1 pad R13: unconnected-(U1D-PR41C-PadR13) -> A11
- U1 pad R14: unconnected-(U1D-PR41B-PadR14) -> A13
- U1 pad R15: unconnected-(U1D-PR38C-PadR15) -> A15
- U1 pad R16: unconnected-(U1D-PR35B-PadR16) -> A16
- U1 pad R7: unconnected-(U1G-PB6A-PadR7) -> A3
- U1 pad R8: unconnected-(U1G-PB13A-PadR8) -> A5
- U1 pad R9: unconnected-(U1G-~{PROGRAM}-PadR9) -> A7
- U1 pad T13: unconnected-(U1D-PR44B-PadT13) -> A10
- U1 pad T14: unconnected-(U1D-PR41D-PadT14) -> A12
- U1 pad T15: unconnected-(U1D-PR38D-PadT15) -> A14
- U1 pad T7: unconnected-(U1G-PB11A-PadT7) -> A2
- U1 pad T8: unconnected-(U1G-PB11B-PadT8) -> A4
- U1 pad T9: unconnected-(U1G-~{INIT}-PadT9) -> A6
- U12 pad A3: /Memory/~{ORAM_CS0} -> /Memory/~{CS}
- U12 pad B1: unconnected-(U12-~{CK}-PadB1) -> GNDD
- U12 pad B2: /Memory/CK -> /Memory/OB_CLKt
- U12 pad B3: unconnected-(U12-VSS-PadB3) -> GNDD
- U12 pad B4: unconnected-(U12-VCC-PadB4) -> +3V3
- U12 pad C1: unconnected-(U12-VSSQ-PadC1) -> GNDD
- U12 pad C3: /Memory/RWDS -> /Memory/OB_RWDS
- U12 pad D1: unconnected-(U12-VCCQ-PadD1) -> +3V3
- U12 pad E4: unconnected-(U12-VCCQ__1-PadE4) -> +3V3
- U12 pad E5: unconnected-(U12-VSSQ__1-PadE5) -> GNDD
- U3 pad 109: unconnected-(U3B-DP2-Pad109) -> Net-(U3B-DP2)
- U3 pad 125: unconnected-(U3B-DP1-Pad125) -> Net-(U3B-DP1)
- U3 pad 13: unconnected-(U3B-~{KEN}-Pad13) -> ~{KEN}
- U3 pad 145: unconnected-(U3B-DP0-Pad145) -> Net-(U3B-DP0)
- U3 pad 16: unconnected-(U3B-HOLD-Pad16) -> HOLD
- U3 pad 17: unconnected-(U3B-AHOLD-Pad17) -> AHOLD
- U3 pad 204: unconnected-(U3B-~{BLAST}-Pad204) -> ~{BLAST}
- U3 pad 26: unconnected-(U3B-HOLDA-Pad26) -> HOLDA
- U3 pad 30: unconnected-(U3B-BREQ-Pad30) -> BREQ
- U3 pad 40: unconnected-(U3B-PWT-Pad40) -> PWT
- U3 pad 41: unconnected-(U3B-PCD-Pad41) -> PCD
- U3 pad 46: unconnected-(U3B-~{EADS}-Pad46) -> ~{EADS}
- U3 pad 49: unconnected-(U3B-~{FLUSH}-Pad49) -> ~{FLUSH}
- U3 pad 5: unconnected-(U3B-~{BRDY}-Pad5) -> ~{BRDY}
- U3 pad 59: unconnected-(U3B-~{SMIACT}-Pad59) -> ~{SMIACT}
- U3 pad 6: unconnected-(U3B-~{BOFF}-Pad6) -> ~{BOFF}
- U3 pad 63: unconnected-(U3B-~{HITM}-Pad63) -> ~{HITM}
- U3 pad 64: unconnected-(U3B-WB~{WT}-Pad64) -> WB~{WT}
- U3 pad 65: unconnected-(U3B-~{SMI}-Pad65) -> ~{SMI}
- U3 pad 70: unconnected-(U3B-~{CACHE}-Pad70) -> ~{CACHE}
- U3 pad 71: unconnected-(U3B-INV-Pad71) -> INV
- U3 pad 73: ~{STPCLK} -> unconnected-(U3B-~{STPCLK}-Pad73)
- U3 pad 90: unconnected-(U3B-DP3-Pad90) -> Net-(U3B-DP3)
Routing:
- net /VideoSubSystem/2A7: track 73.6 -> 0.00 mm, vias 3 -> 0
- net /VideoSubSystem/2A6: track 71.9 -> 0.00 mm, vias 3 -> 0
- net /VideoSubSystem/2A5: track 70.6 -> 0.00 mm, vias 3 -> 0
- net /VideoSubSystem/2A4: track 69.1 -> 0.00 mm, vias 3 -> 0
- net /VideoSubSystem/2A3: track 66.9 -> 0.00 mm, vias 3 -> 0
- net /VideoSubSystem/2A2: track 65.3 -> 0.00 mm, vias 3 -> 0
- net /VideoSubSystem/2A1: track 63.8 -> 0.00 mm, vias 3 -> 0
- net /VideoSubSystem/2A0: track 62.3 -> 0.00 mm, vias 3 -> 0
- net GNDD: track 5.54 -> 59.8 mm, vias 6 -> 27
- net A24: track 0.00 -> 46.5 mm
- net CLK: track 0.00 -> 44.9 mm
- net ~{BE0}: track 0.00 -> 44.1 mm
- net HOLDA: track 0.00 -> 43.7 mm
- net BREQ: track 0.00 -> 43.3 mm
- net RESET: track 0.00 -> 43.2 mm
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Other:
- board size 100 x 170 mm -> 60 x 70 mm
- board text removed: "Address"
- board text removed: "BUS"
- board text removed: "Command"
- board text removed: "Data"
- board text removed: "MEM"
- board text removed: "VID"

Commit message: layout/routing commit
Parts:
- added REF**: C_0201_0603Metric, Capacitor_SMD:C_0201_0603Metric, F.Cu at (37.8, 34.1)
Connections:
- net /Memory/DQ0 renamed /FPGA/DQ0
- net /Memory/DQ1 renamed /FPGA/DQ1
- net /Memory/DQ2 renamed /FPGA/DQ2
- net /Memory/DQ3 renamed /FPGA/DQ3
- net /Memory/DQ4 renamed /FPGA/DQ4
- net /Memory/DQ5 renamed /FPGA/DQ5
- net /Memory/DQ6 renamed /FPGA/DQ6
- net /Memory/DQ7 renamed /FPGA/DQ7
- net /Memory/OB_CLKt renamed /FPGA/OB_CLKt
- net /Memory/OB_RWDS renamed /FPGA/OB_RWDS
- net /Memory/~{RESET} renamed /FPGA/~{RESET}
- U1 pad C10: unconnected-(U1B-PT44B-PadC10) -> D3
- U1 pad C11: unconnected-(U1B-PT49B-PadC11) -> D2
- U1 pad C12: unconnected-(U1B-PT56B-PadC12) -> D1
- U1 pad C13: unconnected-(U1B-PT60B-PadC13) -> D0
- U1 pad D1: unconnected-(U1F-PL8A-PadD1) -> D20
- U1 pad D10: unconnected-(U1B-PT47A-PadD10) -> AHOLD
- U1 pad D11: unconnected-(U1B-PT51A-PadD11) -> A2
- U1 pad D12: unconnected-(U1B-PT58A-PadD12) -> A3
- U1 pad D3: unconnected-(U1F-PL2D-PadD3) -> D19
- U1 pad D4: unconnected-(U1A-PT9B-PadD4) -> ~{LOCK}
- U1 pad D5: unconnected-(U1A-PT13B-PadD5) -> ~{BLAST}
- U1 pad D6: unconnected-(U1A-PT20B-PadD6) -> ~{BOFF}
- U1 pad D7: unconnected-(U1A-PT24B-PadD7) -> ~{BS16}
- U1 pad D8: unconnected-(U1B-PT33B-PadD8) -> ~{BS8}
- U1 pad E1: unconnected-(U1F-PL11D-PadE1) -> D22
- U1 pad E11: unconnected-(U1B-PT51B-PadE11) -> A4
- U1 pad E12: unconnected-(U1B-PT58B-PadE12) -> A5
- U1 pad E2: unconnected-(U1F-PL8B-PadE2) -> D21
- U1 pad E4: unconnected-(U1A-PT9A-PadE4) -> ~{PLOCK}
- U1 pad E5: unconnected-(U1A-PT13A-PadE5) -> ~{ADS}
- U1 pad E6: unconnected-(U1A-PT20A-PadE6) -> ~{RDY}
- U1 pad E7: unconnected-(U1A-PT24A-PadE7) -> ~{KEN}
- U1 pad E8: unconnected-(U1B-PT33A-PadE8) -> HOLD
- U1 pad F1: unconnected-(U1F-PL14A-PadF1) -> D24
- U1 pad F12: unconnected-(U1C-PR8D-PadF12) -> A6
- U1 pad F13: unconnected-(U1C-PR8C-PadF13) -> A7
- U1 pad F2: unconnected-(U1F-PL11C-PadF2) -> D23
- U1 pad G1: unconnected-(U1F-PL20A-PadG1) -> D26
- U1 pad G13: unconnected-(U1C-PR11B-PadG13) -> A8
- U1 pad G15: /Memory/~{CS} -> /FPGA/~{CS}
- U1 pad G2: unconnected-(U1F-PL14B-PadG2) -> D25
- U1 pad H2: unconnected-(U1F-PL20B-PadH2) -> D27
- U1 pad J1: unconnected-(U1F-PL23A-PadJ1) -> D29
- U1 pad J2: unconnected-(U1F-PL23B-PadJ2) -> D28
- U1 pad K1: unconnected-(U1F-PL23C-PadK1) -> D31
- U1 pad K2: unconnected-(U1F-PL23D-PadK2) -> D30
- U1 pad M7: unconnected-(U1G-PB9B-PadM7) -> /FPGA/IO2
- U1 pad N10: unconnected-(U1G-CFG_0-PadN10) -> Net-(JP4-C)
- U1 pad N7: unconnected-(U1G-PB9A-PadN7) -> /FPGA/IO3
- U1 pad N8: unconnected-(U1G-PB15A-PadN8) -> /FPGA/~{CS}
- U1 pad N9: unconnected-(U1G-CCLK-PadN9) -> CCLK
- U1 pad P10: unconnected-(U1G-CFG_1-PadP10) -> Net-(JP5-C)
- U1 pad P9: unconnected-(U1G-DONE-PadP9) -> DONE
- U1 pad R10: A8 -> Net-(JP6-C)
- U1 pad R7: A3 -> unconnected-(U1G-PB6A-PadR7)
- U1 pad R8: A5 -> unconnected-(U1G-PB13A-PadR8)
- U1 pad R9: A7 -> ~{PROGRAM}
- U1 pad T7: A2 -> /FPGA/MISO/IO1
- U1 pad T8: A4 -> /FPGA/MOSI/IO0
- U1 pad T9: A6 -> ~{INIT}
- U12 pad A3: /Memory/~{CS} -> /FPGA/~{CS}
Routing:
- net ~{PLOCK}: track 0.00 -> 55.0 mm, vias 0 -> 2
- net ~{LOCK}: track 0.00 -> 54.8 mm, vias 0 -> 2
- net ~{ADS}: track 0.00 -> 53.7 mm, vias 0 -> 2
- net ~{BLAST}: track 0.00 -> 53.6 mm, vias 0 -> 2
- net ~{BRDY}: track 27.1 -> 51.9 mm, vias 0 -> 2
- net A2: track 70.7 -> 47.0 mm, vias 0 -> 2
- net A3: track 67.8 -> 44.4 mm, vias 0 -> 2
- net ~{BOFF}: track 27.1 -> 50.0 mm, vias 0 -> 2
- net ~{BS16}: track 27.1 -> 49.1 mm, vias 0 -> 2
- net A5: track 65.1 -> 43.9 mm, vias 0 -> 2
- net ~{BS8}: track 27.1 -> 47.9 mm, vias 0 -> 2
- net ~{RDY}: track 27.1 -> 47.9 mm, vias 0 -> 2
- net A7: track 62.3 -> 41.9 mm, vias 0 -> 2
- net A4: track 65.5 -> 45.5 mm, vias 0 -> 2
- net ~{KEN}: track 27.1 -> 46.9 mm, vias 0 -> 2
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