File: PCB/mems.kicad_sch (KiCad schematic)
At the start: 2 parts, among them U10 IS66WVE4M16EBLL-70BLI, U9 IS66WVE4M16EBLL-70BLI

Commit message: more progress
Parts:
- added U12, U13: IS66WVH8M8BLL-100B1LI, IS66WVH8M8ALL-166B1LI:BGA25C100P5X5_800X600X120N, symbol ISSI_OCTAL_PSRAM:IS66WVH8M8ALL-166B1LI
- U10, U9: now not fitted; now left out of the parts list
Connections:
- new net CK: U12.B2 (CK), U13.B2 (CK)
- new net DQ0: U12.D3 (DQ0), U13.D3 (DQ0)
- new net DQ1: U12.D2 (DQ1), U13.D2 (DQ1)
- new net DQ2: U12.C4 (DQ2), U13.C4 (DQ2)
- new net DQ3: U12.D4 (DQ3), U13.D4 (DQ3)
- new net DQ4: U12.D5 (DQ4), U13.D5 (DQ4)
- new net DQ5: U12.E3 (DQ5), U13.E3 (DQ5)
- new net DQ6: U12.E2 (DQ6), U13.E2 (DQ6)
- new net DQ7: U12.E1 (DQ7), U13.E1 (DQ7)
- new net RWDS: U12.C3 (RWDS), U13.C3 (RWDS)
- new net ~{CK}: U13.B1 (~{CK})
- new net ~{ORAM_CS0}: U12.A3 (~{CS})
- new net ~{ORAM_CS1}: U13.A3 (~{CS})
- new net ~{RESET}: U12.A4 (~{RESET}), U13.A4 (~{RESET})

Commit message: route-out in progress
Parts:
- removed U10, U9: IS66WVE4M16EBLL-70BLI, TFBGA48_ISI, symbol 2026-07-26_23-42-22:IS66WVE4M16EBLL-70BLI
- removed U13: IS66WVH8M8BLL-100B1LI, IS66WVH8M8ALL-166B1LI:BGA25C100P5X5_800X600X120N, symbol ISSI_OCTAL_PSRAM:IS66WVH8M8ALL-166B1LI
- added U1: LFE5U-25F-6BG256C, ECP5:BGA256C80P16X16_1400X1400X170, symbol Lattice:LFE5U-25F-6BG256C
- U12: footprint IS66WVH8M8ALL-166B1LI:BGA25C100P5X5_800X600X120N -> Package_BGA:BGA-24_6x8mm_Layout5x5_P1.0mm
Connections:
- net DQ0: now also U1.J15 (PR23B)
- net DQ1: now also U1.J14 (PR20C)
- net DQ2: now also U1.H15 (PR20B)
- net DQ3: now also U1.K16 (PR23C)
- net DQ4: now also U1.J16 (PR23A)
- net DQ5: now also U1.J13 (PR17C)
- net DQ6: now also U1.K14 (PR20D)
- net DQ7: now also U1.K15 (PR23D)
- net ~{RESET}: now also U1.G14 (PR14C)
- net GNDD: now reaches U12.B1 (~{CK})
- net GNDD: now also U12.B3 (VSS), U12.C1 (VSSQ), U12.E5 (VSSQ__1)
- net +3V3: now reaches U12.B4 (VCC)
- net +3V3: now also U12.D1 (VCCQ), U12.E4 (VCCQ__1), U1.H11 (VCCIO2), U1.J11 (VCCIO2)
- net CK renamed OB_CLKt
- net OB_CLKt: now also U1.F16 (PR14A)
- net RWDS renamed OB_RWDS
- net OB_RWDS: now also U1.G16 (PR20A)
- net ~{ORAM_CS0} renamed ~{CS}
- net ~{CS}: now also U1.G15 (PR14B)
- new net A25: U1.F15 (PR11C)
- new net BREQ: U1.C16 (PR5A)
- new net CLK: U1.E15 (PR8B)
- new net HOLDA: U1.D16 (PR8A)
- new net UADDR: U1.E16 (PR11D)
- new net W~{R}: U1.C14 (PR2C)
- new net ~{BE0}: U1.C15 (PR5B)
- new net ~{BE1}: U1.B16 (PR2A)
- new net ~{BE3}: U1.B15 (PR2B)
Other:
- moved on the sheet: U12

Commit message: layout/routing commit
Parts:
- removed U1: LFE5U-25F-6BG256C, ECP5:BGA256C80P16X16_1400X1400X170, symbol Lattice:LFE5U-25F-6BG256C
- removed U12: IS66WVH8M8BLL-100B1LI, Package_BGA:BGA-24_6x8mm_Layout5x5_P1.0mm, symbol ISSI_OCTAL_PSRAM:IS66WVH8M8ALL-166B1LI
