File: PCB/AsicPowerGnd.kicad_sch (KiCad schematic)
At the start: 89 parts, among them U1 LFE5U-25F-6BG256C, U2 TLV62569DBV, U3 AM5x86 PQFP208, U4 TLV62569DBV, U6 TLV62569DBV, U7 AMS1117-2.5, U8 AMS1117-1.2

Commit message: more progress
Parts:
- added J3: ATX-20, Connector_Molex:Molex_Mini-Fit_Jr_5566-20A_2x10_P4.20mm_Vertical, symbol Connector:ATX-20
- C1, C11, C12, C13, C14, C16, C17, C18, C19, C2, C20, C21, C22, C23, C3, C4, L1, L2, R1, R2, R3, R4, U2, U4: now fitted
- JP1: footprint (none) -> Jumper:SolderJumper-2_P1.3mm_Bridged_Pad1.0x1.5mm
- U7, U8: now not fitted; now left out of the parts list
Connections:
- new net: J3.1 (+3.3V), J3.11 (+3.3V), J3.2 (+3.3V)
- new net: J3.13 (GND), J3.15 (GND), J3.16 (GND), J3.17 (GND), J3.3 (GND), J3.5 (GND), J3.7 (GND)
- new net: J3.19 (+5V), J3.20 (+5V), J3.4 (+5V), J3.6 (+5V)

Commit message: more progress
Parts:
- removed U7: AMS1117-2.5, Package_TO_SOT_SMD:SOT-223-3_TabPin2, symbol Regulator_Linear:AMS1117-2.5
- removed U8: AMS1117-1.2, Package_TO_SOT_SMD:SOT-223-3_TabPin2, symbol Regulator_Linear:AMS1117-2.5
- C1, C11, C12, C13, C16, C17, C18, C19, C2, C20, C21, C22, C25, C26, C27, C28, C29, C3, C30, C31, C4, CDC1, CDC10, CDC11, CDC12, CDC13, CDC14, CDC15, CDC16, CDC17, CDC18, CDC19, CDC2, CDC20, CDC21, CDC22, CDC23, CDC24, CDC25, CDC26, CDC27, CDC28, CDC29, CDC3, CDC30, CDC31, CDC32, CDC33, CDC34, CDC35, CDC36, CDC37, CDC38, CDC4, CDC5, CDC6, CDC7, CDC8, CDC9: footprint Capacitor_SMD:C_0402_1005Metric -> (none)
- C10, C14, C15, C23, C24, C32, C33, C5, C6, C7, C8, C9: footprint Capacitor_SMD:C_0603_1608Metric -> (none)
- J3: footprint Connector_Molex:Molex_Mini-Fit_Jr_5566-20A_2x10_P4.20mm_Vertical -> (none)
- JP1: footprint Jumper:SolderJumper-2_P1.3mm_Bridged_Pad1.0x1.5mm -> (none)
- L1, L2, L3: footprint Inductor_SMD:L_1008_2520Metric -> (none)
- R1, R2, R3, R4, R5, R6, R7: footprint Resistor_SMD:R_0402_1005Metric -> (none)

Commit message: route-out in progress
Parts:
- J3: now not fitted; now left out of the parts list
Changed lines of the file:
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@@
 		(unit 1)
 		(body_style 1)
-		(exclude_from_sim no)
-		(in_bom yes)
-		(on_board yes)
-		(in_pos_files yes)
-		(dnp no)
+		(exclude_from_sim yes)
+		(in_bom no)
+		(on_board no)
+		(in_pos_files no)
+		(dnp yes)
 		(fields_autoplaced yes)
 		(property "Reference" "J3"

Commit message: Adding compact fpga on cpu pcb design
Parts:
- renumbered C7 to C1, C2 to C10, C17 to C11, C26 to C12, C3 to C13, C18 to C14, C27 to C15, C4 to C16, C19 to C17, C28 to C18, C11 to C19, C6 to C2, C29 to C21, C12 to C22, C21 to C23, C30 to C24, C13 to C25, C22 to C26, C31 to C27, C14 to C28, C23 to C29, C5 to C3, C32 to C30, C15 to C31, C24 to C32, C10 to C4, C9 to C5, C8 to C6, C1 to C7, C16 to C8, C25 to C9, CDC38 to CDC1, CDC29 to CDC10, CDC28 to CDC11, CDC27 to CDC12, CDC26 to CDC13, CDC25 to CDC14, CDC24 to CDC15, CDC23 to CDC16, CDC22 to CDC17, CDC21 to CDC18, CDC20 to CDC19, CDC37 to CDC2, CDC19 to CDC20, CDC18 to CDC21, CDC17 to CDC22, CDC16 to CDC23, CDC15 to CDC24, CDC14 to CDC25, CDC13 to CDC26, CDC12 to CDC27, CDC11 to CDC28, CDC10 to CDC29, CDC36 to CDC3, CDC9 to CDC30, CDC8 to CDC31, CDC7 to CDC32, CDC6 to CDC33, CDC5 to CDC34, CDC4 to CDC35, CDC3 to CDC36, CDC2 to CDC37, CDC1 to CDC38, CDC35 to CDC4, CDC34 to CDC5, CDC33 to CDC6, CDC32 to CDC7, CDC31 to CDC8, CDC30 to CDC9, J3 to J1, JP1 to JP6, R7 to R10, R5 to R11, R6 to R12, R1 to R6, R2 to R7, R3 to R8, R4 to R9
Connections:
- net Net-(U4-SW): now reaches L2.2, U4.3 (SW)
- net Net-(U4-FB): now reaches C8.2, R8.2, R9.1, U4.5 (FB)
- net Net-(U2-FB): now reaches C7.2, R6.2, R7.1, U2.5 (FB)
- net Net-(U6-FB): now reaches C9.2, R11.2, R12.1, U6.5 (FB)
- net Net-(U2-SW): now reaches L1.2, U2.3 (SW)
- net Net-(U6-SW): now reaches L3.2, U6.3 (SW)
