File: PCB/FPGA.kicad_sch (KiCad schematic)
At the start: 1 part, among them U1 LFE5U-25F-6BG256C

Commit message: progress
Parts:
- removed unit 9 of U1
- U1: footprint LFE5U-25F-6BG256C:BGA256C80P16X16_1400X1400X170 -> ECP5:BGA256C80P16X16_1400X1400X170

Commit message: more progress
Parts:
- removed unit 8 of U1

Commit message: more progress
Parts:
- removed unit 3 of U1
- removed unit 4 of U1
Other:
- note added: "24"
- note added: "32"

Commit message: route-out in progress
Parts:
- removed unit 5 of U1
- added unit 4 of U1
- added Y1: CMOS-50MHz, Oscillator:Oscillator_SMD_Abracon_ASE-4Pin_3.2x2.5mm, symbol Oscillator:ASE-xxxMHz
Connections:
- net VCCIO0 is gone; now on net +3V3: U1.F6 (VCCIO0), U1.F7 (VCCIO0)
- net VCCIO1 is gone; now on net +3V3: U1.F10 (VCCIO1), U1.F11 (VCCIO1)
- net VCCIO7 is gone; now on net +3V3: U1.H6 (VCCIO7), U1.H7 (VCCIO7)
- net ~{CACHE}: now reaches U1.A2 (PT4A)
- net D15: now reaches U1.A3 (PT6A)
- net D14: now reaches U1.A4 (PT6B)
- net ~{SMIACT}: now reaches U1.A5 (PT18A)
- net D13: now reaches U1.A6 (PT18B)
- net D12: now reaches U1.A7 (PT29A)
- net D11: now reaches U1.A8 (PT29B)
- net ~{SMI}: now reaches U1.B3 (PT4B)
- net WB~{WT}: now reaches U1.B4 (PT11B)
- net ~{HITM}: now reaches U1.B5 (PT15B)
- net SRESET: now reaches U1.B6 (PT22B)
- net NMI: now reaches U1.B7 (PT27B)
- net ~{A20M}: now reaches U1.A10 (PT42B)
- net PCD: now reaches U1.A11 (PT53A)
- net PWT: now reaches U1.A12 (PT53B)
- net D~{C}: now reaches U1.A13 (PT65A)
- net D7: now reaches U1.A14 (PT65B)
- net ~{BE2}: now reaches U1.A15 (PT67B)
- net D10: now reaches U1.A9 (PT42A)
- net RESET: now reaches U1.B10 (PT44A)
- net ~{EADS}: now reaches U1.B11 (PT49A)
- net D9: now reaches U1.B12 (PT56A)
- net D8: now reaches U1.B13 (PT60A)
- net M~{IO}: now reaches U1.B14 (PT67A)
- net INTR: now reaches U1.B8 (PT35B)
- net ~{FLUSH}: now reaches U1.B9 (PT38A)
- net D5: now reaches U1.C9 (PT38B)
- net D6: now reaches U1.D9 (PT40A)
- net +3V3: now reaches U1.L6 (VCCIO8)
- net +3V3: now also U1.K11 (VCCIO3), U1.L11 (VCCIO3), Y1.1 (EN), Y1.4 (Vdd)
- net CFG_0: now reaches U1.N10 (CFG_0)
- net CCLK: now reaches U1.N9 (CCLK)
- net CFG_1: now reaches U1.P10 (CFG_1)
- net DONE: now reaches U1.P9 (DONE)
- net CFG_2: now reaches U1.R10 (CFG_2)
- net A3: now reaches U1.R7 (PB6A)
- net A5: now reaches U1.R8 (PB13A)
- net ~{PROGRAM}: now reaches U1.R9 (~{PROGRAM})
- net A2: now reaches U1.T7 (PB11A)
- net A4: now reaches U1.T8 (PB11B)
- net ~{INIT}: now reaches U1.T9 (~{INIT})
- net D16: now reaches U1.B1 (PL2A)
- net INV: now reaches U1.B2 (PL2B)
- net D18: now reaches U1.C1 (PL5A)
- net D17: now reaches U1.C2 (PL5B)
- new net A10: U1.T13 (PR44B)
- new net A11: U1.R13 (PR41C)
- new net A12: U1.T14 (PR41D)
- new net A13: U1.R14 (PR41B)
- new net A14: U1.T15 (PR38D)
- new net A15: U1.R15 (PR38C)
- new net A16: U1.R16 (PR35B)
- new net A17: U1.P15 (PR32B)
- new net A18: U1.P16 (PR35A)
- new net A19: U1.N14 (PR35D)
- new net A20: U1.N16 (PR32A)
- new net A21: U1.M15 (PR26D)
- new net A22: U1.M16 (PR26C)
- new net A23: U1.L15 (PR26B)
- new net A24: U1.L16 (PR26A)
- new net A9: U1.R12 (PR44A)
- new net GNDD: Y1.2 (GND)
- new net LRC_GPLL0T_IN: U1.P11 (PR47C), Y1.3 (OUT)
Other:
- moved on the sheet: U1B, U1G

Commit message: layout/routing commit
Parts:
- added JP2: O:Ena/C:Dis, symbol Jumper:SolderJumper_2_Open
- added JP3: O:3x/C:4x, symbol Jumper:SolderJumper_2_Open
- added JP4: C0, symbol Jumper:SolderJumper_3_Bridged12
- added JP5: C1, symbol Jumper:SolderJumper_3_Bridged12
- added JP6: C2, symbol Jumper:SolderJumper_3_Bridged12
- added R14, R15, R16, R17, R18: 10k, symbol Device:R_Small
- added unit 3 of U1
- added unit 8 of U1
- added U12: IS66WVH8M8BLL-100B1LI, Package_BGA:BGA-24_6x8mm_Layout5x5_P1.0mm, symbol ISSI_OCTAL_PSRAM:IS66WVH8M8ALL-166B1LI
- added U18: 4068, Package_SO:TSSOP-14_4.4x5mm_P0.65mm, symbol 4xxx_IEEE:4068
- added U3: AM5x86 PQFP208, Package_QFP:LQFP-208_28x28mm_P0.5mm, symbol am5x86:am5x86
Connections:
- net +3V3: now also JP4.3 (B), JP5.1 (A), JP6.3 (B), U1.H11 (VCCIO2), U1.J11 (VCCIO2), U12.B4 (VCC), U12.D1 (VCCQ), U12.E4 (VCCQ__1), U18.14 (Vdd)
- net A10: now also U3.186 (A10)
- net A11: now also U3.182 (A11)
- net A12: now also U3.180 (A12)
- net A13: now also U3.178 (A13)
- net A14: now also U3.177 (A14)
- net A15: now also U3.174 (A15)
- net A16: now also U3.173 (A16)
- net A17: now also U3.171 (A17)
- net A18: now also U3.166 (A18)
- net A19: now also U3.165 (A19)
- net A2: now also U1.D11 (PT51A), U3.202 (A2); no longer U1.T7 (PB11A)
- net A20: now also U3.164 (A20)
- net A21: now also U3.161 (A21)
- net A22: now also U3.160 (A22)
- net A23: now also U3.159 (A23)
- net A24: now also U18.2 (A), U3.158 (A24)
- net A3: now also U1.D12 (PT58A), U3.197 (A3); no longer U1.R7 (PB6A)
- net A4: now also U1.E11 (PT51B), U3.196 (A4); no longer U1.T8 (PB11B)
- net A5: now also U1.E12 (PT58B), U3.195 (A5); no longer U1.R8 (PB13A)
- net A9: now also U3.187 (A9)
- net D10: now also U3.119 (D10)
- net D11: now also U3.118 (D11)
- net D12: now also U3.117 (D12)
- net D13: now also U3.116 (D13)
- net D14: now also U3.113 (D14)
- net D15: now also U3.112 (D15)
- net D16: now also U3.108 (D16)
- net D17: now also U3.103 (D17)
- net D18: now also U3.101 (D18)
- net D5: now also U3.130 (D5)
- net D6: now also U3.129 (D6)
- net D7: now also U3.126 (D7)
- net D8: now also U3.124 (D8)
- net D9: now also U3.123 (D9)
- net D~{C}: now also U3.39 (D~{C})
- net GNDD: now also JP2.1 (A), JP3.1 (A), JP4.1 (A), JP5.3 (B), JP6.1 (A), U12.B1 (~{CK}), U12.B3 (VSS), U12.C1 (VSSQ), U12.E5 (VSSQ__1), U18.7 (Vss)
- net INTR: now also U3.50 (INTR)
- net INV: now also U3.71 (INV)
- net M~{IO}: now also U3.37 (M~{IO})
- net NMI: now also U3.51 (NMI)
- net PCD: now also U3.41 (PCD)
- net PWT: now also U3.40 (PWT)
- net RESET: now also U3.48 (RESET)
- net SRESET: now also U3.58 (SRESET)
- net WB~{WT}: now also U3.64 (WB~{WT})
- net ~{A20M}: now also U3.47 (~{A20M})
- net ~{BE2}: now also U3.33 (~{BE2})
- net ~{CACHE}: now also U3.70 (~{CACHE})
- net ~{EADS}: now also U3.46 (~{EADS})
- net ~{FLUSH}: now also U3.49 (~{FLUSH})
- net ~{HITM}: now also U3.63 (~{HITM})
- net ~{SMIACT}: now also U3.59 (~{SMIACT})
- net ~{SMI}: now also U3.65 (~{SMI})
- net D3: now reaches U1.C10 (PT44B)
- net D3: now also U3.141 (D3)
- net D2: now reaches U1.C11 (PT49B)
- net D2: now also U3.142 (D2)
- net D1: now reaches U1.C12 (PT56B)
- net D1: now also U3.143 (D1)
- net D0: now reaches U1.C13 (PT60B)
- net D0: now also U3.144 (D0)
- net AHOLD: now reaches U1.D10 (PT47A)
- net AHOLD: now also U3.17 (AHOLD)
- net ~{BS8}: now reaches U1.D8 (PT33B)
- net ~{BS8}: now also U3.8 (~{BS8})
- net HOLD: now reaches U1.E8 (PT33A)
- net HOLD: now also U3.16 (HOLD)
- net IO2: now reaches U1.M7 (PB9B)
- net IO3: now reaches U1.N7 (PB9A)
- net ~{CS}: now reaches U1.N8 (PB15A)
- net ~{CS}: now also U1.G15 (PR14B), U12.A3 (~{CS})
- net D20: now reaches U1.D1 (PL8A)
- net D20: now also U3.99 (D20)
- net D19: now reaches U1.D3 (PL2D)
- net D19: now also U3.100 (D19)
- net D22: now reaches U1.E1 (PL11D)
- net D22: now also U3.92 (D22)
- net D21: now reaches U1.E2 (PL8B)
- net D21: now also U3.93 (D21)
- net D24: now reaches U1.F1 (PL14A)
- net D24: now also U3.87 (D24)
- net D23: now reaches U1.F2 (PL11C)
- net D23: now also U3.91 (D23)
- net D26: now reaches U1.G1 (PL20A)
- net D26: now also U3.84 (D26)
- net D25: now reaches U1.G2 (PL14B)
- net D25: now also U3.85 (D25)
- net D27: now reaches U1.H2 (PL20B)
- net D27: now also U3.83 (D27)
- net D29: now reaches U1.J1 (PL23A)
- net D29: now also U3.78 (D29)
- net D28: now reaches U1.J2 (PL23B)
- net D28: now also U3.79 (D28)
- net D31: now reaches U1.K1 (PL23C)
- net D31: now also U3.74 (D31)
- net D30: now reaches U1.K2 (PL23D)
- net D30: now also U3.75 (D30)
- net ~{LOCK}: now reaches U1.D4 (PT9B)
- net ~{LOCK}: now also U3.207 (~{LOCK})
- net ~{BLAST}: now reaches U1.D5 (PT13B)
- net ~{BLAST}: now also U3.204 (~{BLAST})
- net ~{BOFF}: now reaches U1.D6 (PT20B)
- net ~{BOFF}: now also U3.6 (~{BOFF})
- net ~{BS16}: now reaches U1.D7 (PT24B)
- net ~{BS16}: now also U3.7 (~{BS16})
- net ~{PLOCK}: now reaches U1.E4 (PT9A)
- net ~{PLOCK}: now also U3.206 (~{PLOCK})
- net ~{ADS}: now reaches U1.E5 (PT13A)
- net ~{ADS}: now also U3.203 (~{ADS})
- net ~{RDY}: now reaches U1.E6 (PT20A)
- net ~{RDY}: now also U3.12 (~{RDY})
- net ~{KEN}: now reaches U1.E7 (PT24A)
- net ~{KEN}: now also U3.13 (~{KEN})
- net CFG_0: no longer names the net of U1.N10 (CFG_0)
- net CFG_0: now also JP4.2 (C)
- net CFG_1: no longer names the net of U1.P10 (CFG_1)
- net CFG_1: now also JP5.2 (C)
- net CFG_2: no longer names the net of U1.R10 (CFG_2)
- net CFG_2: now also JP6.2 (C)
- new net: R17.2, U3.109 (DP2)
- new net: R18.2, U3.90 (DP3)
- new net: JP2.2 (B), R14.2, U3.194 (~{UP})
- new net: JP3.2 (B), U3.11 (CLKMUL)
- new net: R16.2, U3.125 (DP1)
- new net: R15.2, U3.145 (DP0)
- new net: U1.M10 (TDO), U3.168 (TDI)
- new net +3.3V: R14.1, R15.1, R16.1, R17.1, R18.1
- new net A25: U1.F15 (PR11C), U18.3 (B), U3.154 (A25)
- new net A26: U18.5 (D), U3.153 (A26)
- new net A27: U18.4 (C), U3.152 (A27)
- new net A28: U18.12 (H), U3.151 (A28)
- new net A29: U18.11 (G), U3.149 (A29)
- new net A30: U18.10 (F), U3.148 (A30)
- new net A31: U18.9 (E), U3.147 (A31)
- new net A6: U1.F12 (PR8D), U3.193 (A6)
- new net A7: U1.F13 (PR8C), U3.192 (A7)
- new net A8: U1.G13 (PR11B), U3.190 (A8)
- new net BREQ: U1.C16 (PR5A), U3.30 (BREQ)
- new net CLK: U1.E15 (PR8B), U3.24 (CLK)
- new net D4: U3.140 (D4)
- new net DQ0: U1.J15 (PR23B), U12.D3 (DQ0)
- new net DQ1: U1.J14 (PR20C), U12.D2 (DQ1)
- new net DQ2: U1.H15 (PR20B), U12.C4 (DQ2)
- new net DQ3: U1.K16 (PR23C), U12.D4 (DQ3)
- new net DQ4: U1.J16 (PR23A), U12.D5 (DQ4)
- new net DQ5: U1.J13 (PR17C), U12.E3 (DQ5)
- new net DQ6: U1.K14 (PR20D), U12.E2 (DQ6)
- new net DQ7: U1.K15 (PR23D), U12.E1 (DQ7)
- new net HOLDA: U1.D16 (PR8A), U3.26 (HOLDA)
- new net MISO/IO1: U1.T7 (PB11A)
- new net MOSI/IO0: U1.T8 (PB11B)
- new net OB_CLKt: U1.F16 (PR14A), U12.B2 (CK)
- new net OB_RWDS: U1.G16 (PR20A), U12.C3 (RWDS)
- new net TCK: U1.T10 (TCK), U3.18 (TCK)
- new net TDI: U1.R11 (TDI)
- new net TDO: U3.68 (TDO)
- new net TMS: U1.T11 (TMS), U3.167 (TMS)
- new net UADDR: U1.E16 (PR11D), U18.1 (K)
- new net W~{R}: U1.C14 (PR2C), U3.27 (W~{R})
- new net ~{BE0}: U1.C15 (PR5B), U3.31 (~{BE0})
- new net ~{BE1}: U1.B16 (PR2A), U3.32 (~{BE1})
- new net ~{BE3}: U1.B15 (PR2B), U3.34 (~{BE3})
- new net ~{BRDY}: U3.5 (~{BRDY})
- new net ~{RESET}: U1.G14 (PR14C), U12.A4 (~{RESET})
- new net ~{UADDR}: U18.13 (J)
- no-connect marks 0 -> 4
Other:
- note added: "36"
- note added: "Slave SPI =001 Slave Serial =101 Slave Parallel =111 Master SPI SERIAL =010"
- note added: "pin saver option. Reduces address space to 16MB"
- moved on the sheet: U1F, U1G

Commit message: Adding compact fpga on cpu pcb design
Parts:
- renumbered JP6 to JP1, JP5 to JP2, JP4 to JP3, JP2 to JP4, JP3 to JP5, R14 to R1, R15 to R2, R16 to R3, R17 to R4, R18 to R5
Connections:
- net +3V3: no longer JP1.3 (B)
- net A10: now also U1.H3 (PL14D); no longer U1.T13 (PR44B)
- net A11: now also U1.J3 (PL20C); no longer U1.R13 (PR41C)
- net A12: now also U1.J4 (PL17C)
- net A13: now also U1.K3 (PL20D); no longer U1.R14 (PR41B)
- net A14: now also U1.H2 (PL20B); no longer U1.T15 (PR38D)
- net A15: now also U1.H5 (PL17A), U1.J2 (PL23B); no longer U1.R15 (PR38C)
- net A16: now also U1.J5 (PL17D); no longer U1.R16 (PR35B)
- net A17: now also U1.J1 (PL23A); no longer U1.P15 (PR32B)
- net A18: now also U1.K2 (PL23D); no longer U1.P16 (PR35A)
- net A19: now also U1.K1 (PL23C); no longer U1.N14 (PR35D)
- net A2: now also U1.D3 (PL2D); no longer U1.D11 (PT51A)
- net A20: no longer U1.N16 (PR32A)
- net A3: now also U1.E4 (PT9A); no longer U1.D12 (PT58A)
- net A4: now also U1.E3 (PL5C)
- net A5: now also U1.F4 (PL8C)
- net A6: now also U1.F3 (PL5D)
- net A7: now also U1.G4 (PL11B); no longer U1.F13 (PR8C)
- net A8: now also U1.G2 (PL14B), U1.G3 (PL14C); no longer U1.G13 (PR11B)
- net A9: now also U1.H4 (PL17B); no longer U1.R12 (PR44A)
- net AHOLD: now also U1.C8 (PT35A); no longer U1.D10 (PT47A)
- net BREQ: now also U1.C10 (PT44B); no longer U1.C16 (PR5A)
- net CLK: now also U1.D9 (PT40A)
- net D0: no longer U1.C13 (PT60B)
- net D1: no longer U1.C12 (PT56B)
- net D10: now also U1.P12 (PR47D), U1.P7 (PB6B)
- net D11: now also U1.N12 (PR44D), U1.R7 (PB6A)
- net D12: now also U1.P8 (PB13B), U1.T13 (PR44B)
- net D13: now also U1.M8 (PB15B), U1.R13 (PR41C)
- net D14: now also U1.M9 (PB18A), U1.P13 (PR41A)
- net D15: now also U1.N13 (PR38A)
- net D16: now also U1.R14 (PR41B)
- net D17: now also U1.T15 (PR38D)
- net D18: now also U1.P14 (PR38B)
- net D19: now also U1.N14 (PR35D); no longer U1.D3 (PL2D)
- net D2: no longer U1.C11 (PT49B)
- net D20: now also U1.M13 (PR35C), U1.R15 (PR38C)
- net D21: now also U1.R16 (PR35B)
- net D22: now also U1.P15 (PR32B)
- net D23: now also U1.P16 (PR35A)
- net D24: now also U1.N16 (PR32A)
- net D25: now also U1.L13 (PR29C); no longer U1.G2 (PL14B)
- net D26: now also U1.K13 (PR29A)
- net D27: now also U1.K12 (PR29B); no longer U1.H2 (PL20B)
- net D28: now also U1.J12 (PR17D); no longer U1.J2 (PL23B)
- net D29: now also U1.H14 (PR14D); no longer U1.J1 (PL23A)
- net D3: no longer U1.C10 (PT44B)
- net D30: now also U1.H13 (PR17B); no longer U1.K2 (PL23D)
- net D31: no longer U1.K1 (PL23C)
- net D4: now also U1.R6 (PB4B)
- net D5: now also U1.T6 (PB4A); no longer U1.C9 (PT38B)
- net D6: now also U1.M11 (PR47A); no longer U1.D9 (PT40A)
- net D7: now also U1.N11 (PR47B)
- net D8: now also U1.M12 (PR44C)
- net D9: now also U1.R12 (PR44A)
- net D~{C}: now also U1.C13 (PT60B)
- net HOLD: now also U1.D8 (PT33B)
- net HOLDA: now also U1.C9 (PT38B); no longer U1.D16 (PR8A)
- net INTR: now also U1.B16 (PR2A)
- net INV: now also U1.G14 (PR14C)
- net M~{IO}: now also U1.D13 (PT62A); no longer U1.B14 (PT67A)
- net NMI: now also U1.C16 (PR5A)
- net PCD: now also U1.C14 (PR2C)
- net PWT: now also U1.D14 (PR2D)
- net RESET: now also U1.C15 (PR5B)
- net SRESET: now also U1.D16 (PR8A)
- net WB~{WT}: now also U1.F13 (PR8C)
- net W~{R}: now also U1.D10 (PT47A); no longer U1.C14 (PR2C)
- net ~{A20M}: now also U1.A15 (PT67B)
- net ~{ADS}: now also U1.D4 (PT9B)
- net ~{BE0}: now also U1.D11 (PT51A); no longer U1.C15 (PR5B)
- net ~{BE1}: now also U1.C11 (PT49B); no longer U1.B16 (PR2A)
- net ~{BE2}: now also U1.D12 (PT58A); no longer U1.A15 (PT67B)
- net ~{BE3}: now also U1.C12 (PT56B); no longer U1.B15 (PR2B)
- net ~{BLAST}: no longer U1.D5 (PT13B)
- net ~{BOFF}: now also U1.C5 (PT15A); no longer U1.D6 (PT20B)
- net ~{BRDY}: now also U1.D5 (PT13B)
- net ~{BS16}: now also U1.D6 (PT20B); no longer U1.D7 (PT24B)
- net ~{BS8}: now also U1.C6 (PT22A); no longer U1.D8 (PT33B)
- net ~{CACHE}: now also U1.G13 (PR11B)
- net ~{EADS}: now also U1.B14 (PT67A)
- net ~{FLUSH}: now also U1.B15 (PR2B)
- net ~{HITM}: now also U1.E14 (PR5C)
- net ~{KEN}: now also U1.C7 (PT27A)
- net ~{LOCK}: now also U1.C4 (PT11A); no longer U1.D4 (PT9B)
- net ~{PLOCK}: now also U1.C3 (PL2C); no longer U1.E4 (PT9A)
- net ~{RDY}: now also U1.D7 (PT24B)
- net ~{RESET}: no longer U1.G14 (PR14C)
- net ~{SMIACT}: now also U1.E13 (PT62B)
- net ~{SMI}: now also U1.F14 (PR5D)
- net Net-(U3B-DP2): now reaches R4.2, U3.109 (DP2)
- net unconnected-(U1B-PT47B-PadE10): now reaches U1.E10 (PT47B)
- net unconnected-(U1B-PT40B-PadE9): now reaches U1.E9 (PT40B)
- net Net-(U3B-DP3): now reaches R5.2, U3.90 (DP3)
- net Net-(JP4-C): now reaches JP3.2 (C), U1.N10 (CFG_0)
- net Net-(JP5-C): now reaches JP2.2 (C), U1.P10 (CFG_1)
- net Net-(JP6-C): now reaches JP1.2 (C), U1.R10 (CFG_2)
- net unconnected-(U1G-PB13A-PadR8): now reaches U1.R8 (PB13A)
- net Net-(JP2-B): now reaches JP4.2 (B), R1.2, U3.194 (~{UP})
- net Net-(JP3-B): now reaches JP5.2 (B), U3.11 (CLKMUL)
- net unconnected-(U1F-PL8D-PadF5): now reaches U1.F5 (PL8D)
- net unconnected-(U1F-PL11A-PadG5): now reaches U1.G5 (PL11A)
- net unconnected-(U1C-PR11A-PadG12): now reaches U1.G12 (PR11A)
- net unconnected-(U1C-PR17A-PadH12): now reaches U1.H12 (PR17A)
- net Net-(U3B-DP1): now reaches R3.2, U3.125 (DP1)
- net unconnected-(U3B-NC-Pad127): now reaches U3.127 (NC)
- net Net-(U3B-DP0): now reaches R2.2, U3.145 (DP0)
- net Net-(U1H-TDO): now reaches U1.M10 (TDO), U3.168 (TDI)
- net unconnected-(U3B-NC-Pad3): now reaches U3.3 (NC)
- net unconnected-(U3B-~{PCHK}-Pad4): now reaches U3.4 (~{PCHK})
- net unconnected-(U3B-~{FERR}-Pad66): now reaches U3.66 (~{FERR})
- net unconnected-(U3B-NC-Pad67): now reaches U3.67 (NC)
- net unconnected-(U3B-~{IGNNE}-Pad72): now reaches U3.72 (~{IGNNE})
- net unconnected-(U3B-~{STPCLK}-Pad73): now reaches U3.73 (~{STPCLK})
- net unconnected-(U3B-NC-Pad96): now reaches U3.96 (NC)
- net unconnected-(U18-NC-Pad6): now reaches U18.6 (NC)
- net unconnected-(U18-NC-Pad8): now reaches U18.8 (NC)
- net unconnected-(U1D-PR29D-PadL12): now reaches U1.L12 (PR29D)
- net unconnected-(U1D-PR32C-PadL14): now reaches U1.L14 (PR32C)
- net unconnected-(U1D-PR32D-PadM14): now reaches U1.M14 (PR32D)
