File: PCB/am5x86.kicad_sch (KiCad schematic)
At the start: 45 parts

Commit message: progress
Parts:
- removed C10, C5, C6, C7, C8, C9: 47uF, Capacitor_SMD:C_0603_1608Metric, symbol Device:C_Small
- removed CDC1, CDC10, CDC11, CDC12, CDC13, CDC14, CDC15, CDC16, CDC17, CDC18, CDC19, CDC2, CDC20, CDC21, CDC22, CDC23, CDC24, CDC25, CDC26, CDC27, CDC28, CDC29, CDC3, CDC30, CDC31, CDC32, CDC33, CDC34, CDC35, CDC36, CDC37, CDC38, CDC4, CDC5, CDC6, CDC7, CDC8, CDC9: 1uF, Capacitor_SMD:C_0402_1005Metric, symbol Device:C_Small
- removed unit 1 of U3
- U3: value (none) -> AM5x86 PQFP208

Commit message: more progress
Parts:
- added U1: LFE5U-25F-6BG256C, ECP5:BGA256C80P16X16_1400X1400X170, symbol Lattice:LFE5U-25F-6BG256C
Connections:
- net TMS: now reaches U3.167 (TMS)
- net TMS: now also U1.T11 (TMS)
- net at U3.168 (TDI): now also U1.M10 (TDO)
- net TCK: now reaches U3.18 (TCK)
- net TCK: now also U1.T10 (TCK)
- net TDO: now reaches U3.68 (TDO)
- new net TDI: U1.R11 (TDI)

Commit message: more progress
Parts:
- added unit 3 of U1
- added unit 4 of U1
Connections:
- new net VCCIO2: U1.H11 (VCCIO2), U1.J11 (VCCIO2)
- new net VCCIO3: U1.K11 (VCCIO3), U1.L11 (VCCIO3)

Commit message: started initial layout
Connections:
- net CLKMUL: now reaches U3.11 (CLKMUL)
- net ~{RDY_CPU}: now reaches U3.12 (~{RDY})
- net ~{ADS_CPU}: now reaches U3.203 (~{ADS})
- net ~{PLOCK}: now reaches U3.206 (~{PLOCK})
- net ~{LOCK}: now reaches U3.207 (~{LOCK})
- net CLK_CPU: now reaches U3.24 (CLK)
- net W~{R}: now reaches U3.27 (W~{R})
- net ~{BE0}: now reaches U3.31 (~{BE0})
- net ~{BE1}: now reaches U3.32 (~{BE1})
- net ~{BE2}: now reaches U3.33 (~{BE2})
- net ~{BE3}: now reaches U3.34 (~{BE3})
- net M~{IO}: now reaches U3.37 (M~{IO})
- net D~{C}: now reaches U3.39 (D~{C})
- net ~{A20M}: now reaches U3.47 (~{A20M})
- net ~{BS16}: now reaches U3.7 (~{BS16})
- net ~{STPCLK}: now reaches U3.73 (~{STPCLK})
- net ~{BS8}: now reaches U3.8 (~{BS8})

Commit message: More layout work
Connections:
- net ~{UP}: now reaches U3.194 (~{UP})
- net RESET: now reaches U3.48 (RESET)
- net INTR: now reaches U3.50 (INTR)
- net NMI: now reaches U3.51 (NMI)
- net SRESET: now reaches U3.58 (SRESET)
- net CLK_CPU renamed CLK
- net ~{ADS_CPU} renamed ~{ADS}
- net ~{RDY_CPU} renamed ~{RDY}

Commit message: route-out in progress
Parts:
- removed unit 3 of U1
- removed unit 4 of U1
- added JP2: O:Ena/C:Dis, symbol Jumper:SolderJumper_2_Open
- added JP3: O:3x/C:4x, symbol Jumper:SolderJumper_2_Open
- added R14, R15, R16, R17, R18: 10k, symbol Device:R_Small
- added U18: 4068, Package_SO:TSSOP-14_4.4x5mm_P0.65mm, symbol 4xxx_IEEE:4068
Connections:
- net A24: now also U18.2 (A)
- net A25: now also U18.3 (B)
- net A26: now also U18.5 (D)
- net A27: now also U18.4 (C)
- net A28: now also U18.12 (H)
- net A29: now also U18.11 (G)
- net A30: now also U18.10 (F)
- net A31: now also U18.9 (E)
- net at U3.109 (DP2): now also R17.2
- net at U3.125 (DP1): now also R16.2
- net ~{KEN}: now reaches U3.13 (~{KEN})
- net at U3.145 (DP0): now also R15.2
- net HOLD: now reaches U3.16 (HOLD)
- net AHOLD: now reaches U3.17 (AHOLD)
- net ~{BLAST}: now reaches U3.204 (~{BLAST})
- net HOLDA: now reaches U3.26 (HOLDA)
- net BREQ: now reaches U3.30 (BREQ)
- net PWT: now reaches U3.40 (PWT)
- net PCD: now reaches U3.41 (PCD)
- net ~{EADS}: now reaches U3.46 (~{EADS})
- net ~{FLUSH}: now reaches U3.49 (~{FLUSH})
- net ~{BRDY}: now reaches U3.5 (~{BRDY})
- net ~{SMIACT}: now reaches U3.59 (~{SMIACT})
- net ~{BOFF}: now reaches U3.6 (~{BOFF})
- net ~{HITM}: now reaches U3.63 (~{HITM})
- net WB~{WT}: now reaches U3.64 (WB~{WT})
- net ~{SMI}: now reaches U3.65 (~{SMI})
- net ~{CACHE}: now reaches U3.70 (~{CACHE})
- net INV: now reaches U3.71 (INV)
- net at U3.90 (DP3): now also R18.2
- net CLKMUL: no longer names the net of U3.11 (CLKMUL)
- net CLKMUL: now also JP3.2 (B)
- net ~{STPCLK}: no longer names the net of U3.73 (~{STPCLK})
- net ~{UP}: no longer names the net of U3.194 (~{UP})
- net ~{UP}: now also JP2.2 (B), R14.2
- new net +3.3V: R14.1, R15.1, R16.1, R17.1, R18.1
- new net +3V3: U18.14 (Vdd)
- new net GNDD: JP2.1 (A), JP3.1 (A), U18.7 (Vss)
- new net UADDR: U18.1 (K)
- new net ~{UADDR}: U18.13 (J)
- no-connect marks 0 -> 4
Other:
- note added: "36"
- note added: "pin saver option. Reduces address space to 16MB"
- moved on the sheet: U1H

Commit message: Adding compact fpga on cpu pcb design
Parts:
- renumbered JP2 to JP7, JP3 to JP8, R14 to R13, R15 to R14, R16 to R15, R17 to R16, R18 to R17, U1 to U10, U3 to U8, U18 to U9
Changed lines of the file:
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@@
 		(dnp no)
 		(fields_autoplaced yes)
-		(property "Reference" "R14"
+		(property "Reference" "R13"
 			(at 166.37 30.4799 0)
 			(show_name no)
@@
 			(project "Poor86"
 				(path "/516eb290-d08d-4e43-95ba-5c21610df4ad/332916af-3e11-4b31-930a-ff884aaa5dd6"
-					(reference "R14")
+					(reference "R13")
 					(unit 1)
 				)
@@
 		(in_pos_files yes)
 		(dnp no)
-		(property "Reference" "JP2"
+		(property "Reference" "JP7"
 			(at 166.624 41.91 90)
 			(show_name no)
@@
 			(project "Poor86"
 				(path "/516eb290-d08d-4e43-95ba-5c21610df4ad/332916af-3e11-4b31-930a-ff884aaa5dd6"
-					(reference "JP2")
+					(reference "JP7")
 					(unit 1)
 				)
@@
 		(dnp no)
 		(fields_autoplaced yes)
-		(property "Reference" "#PWR096"
+		(property "Reference" "#PWR093"
 			(at 163.83 53.34 0)
 			(hide yes)
@@
 			(project "Poor86"
 				(path "/516eb290-d08d-4e43-95ba-5c21610df4ad/332916af-3e11-4b31-930a-ff884aaa5dd6"
-					(reference "#PWR096")
+					(reference "#PWR093")
 					(unit 1)
 				)
@@
 		(in_pos_files yes)
 		(dnp no)
-		(property "Reference" "#PWR094"
+		(property "Reference" "#PWR090"
 			(at 152.4 162.56 0)
 			(hide yes)
@@
 			(project "Poor86"
 				(path "/516eb290-d08d-4e43-95ba-5c21610df4ad/332916af-3e11-4b31-930a-ff884aaa5dd6"
-					(reference "#PWR094")
+					(reference "#PWR090")
 					(unit 1)
 				)
@@
 		(in_pos_files yes)
 		(dnp no)
-		(property "Reference" "#PWR099"
+		(property "Reference" "#PWR095"
 			(at 248.92 22.86 0)
 			(hide yes)
@@
 			(project "Poor86"
 				(path "/516eb290-d08d-4e43-95ba-5c21610df4ad/332916af-3e11-4b31-930a-ff884aaa5dd6"
-					(reference "#PWR099")
+					(reference "#PWR095")
 					(unit 1)
 				)
@@
 		(dnp no)
 		(fields_autoplaced yes)
-		(property "Reference" "U3"
+		(property "Reference" "U8"
 			(at 30.734 105.918 0)
 			(hide yes)
@@
 			(project "Poor86"
 				(path "/516eb290-d08d-4e43-95ba-5c21610df4ad/332916af-3e11-4b31-930a-ff884aaa5dd6"
-					(reference "U3")
+					(reference "U8")
 					(unit 3)
 				)
@@
 		(in_pos_files yes)
 		(dnp no)
-		(property "Reference" "R17"
+		(property "Reference" "R16"
 			(at 256.54 24.13 0)
 			(show_name no)
@@
 			(project "Poor86"
 				(path "/516eb290-d08d-4e43-95ba-5c21610df4ad/332916af-3e11-4b31-930a-ff884aaa5dd6"
-					(reference "R17")
+					(reference "R16")
 					(unit 1)
 				)
@@
 		(dnp no)
 		(fields_autoplaced yes)
-		(property "Reference" "#PWR098"
+		(property "Reference" "#PWR094"
 			(at 175.26 53.34 0)
 			(hide yes)
@@
 			(project "Poor86"
 				(path "/516eb290-d08d-4e43-95ba-5c21610df4ad/332916af-3e11-4b31-930a-ff884aaa5dd6"
-					(reference "#PWR098")
+					(reference "#PWR094")
 					(unit 1)
 				)
@@
 		(dnp no)
 		(fields_autoplaced yes)
-		(property "Reference" "#PWR097"
+		(property "Reference" "#PWR092"
 			(at 163.83 33.02 0)
 			(hide yes)
@@
 			(project "Poor86"
 				(path "/516eb290-d08d-4e43-95ba-5c21610df4ad/332916af-3e11-4b31-930a-ff884aaa5dd6"
-					(reference "#PWR097")
+					(reference "#PWR092")
 					(unit 1)
 				)
@@
 		(in_pos_files yes)
 		(dnp no)
-		(property "Reference" "R15"
+		(property "Reference" "R14"
 			(at 256.54 19.05 0)
 			(show_name no)
@@
 			(project "Poor86"
 				(path "/516eb290-d08d-4e43-95ba-5c21610df4ad/332916af-3e11-4b31-930a-ff884aaa5dd6"
-					(reference "R15")
+					(reference "R14")
 					(unit 1)
 				)
@@
 		(dnp no)
 		(fields_autoplaced yes)
-		(property "Reference" "U3"
+		(property "Reference" "U8"
 			(at 195.834 136.398 0)
 			(hide yes)
@@
 			(project "Poor86"
 				(path "/516eb290-d08d-4e43-95ba-5c21610df4ad/332916af-3e11-4b31-930a-ff884aaa5dd6"
-					(reference "U3")
+					(reference "U8")
 					(unit 2)
 				)
@@
 		(in_pos_files yes)
 		(dnp no)
-		(property "Reference" "R16"
+		(property "Reference" "R15"
 			(at 256.54 21.59 0)
 			(show_name no)
@@
 			(project "Poor86"
 				(path "/516eb290-d08d-4e43-95ba-5c21610df4ad/332916af-3e11-4b31-930a-ff884aaa5dd6"
-					(reference "R16")
+					(reference "R15")
 					(unit 1)
 				)
@@
 		(dnp no)
 		(fields_autoplaced yes)
-		(property "Reference" "U18"
+		(property "Reference" "U9"
 			(at 154.5433 158.75 0)
 			(show_name no)
@@
 			(project "Poor86"
 				(path "/516eb290-d08d-4e43-95ba-5c21610df4ad/332916af-3e11-4b31-930a-ff884aaa5dd6"
-					(reference "U18")
+					(reference "U9")
 					(unit 1)
 				)
@@
 		(dnp no)
 		(fields_autoplaced yes)
-		(property "Reference" "#PWR095"
+		(property "Reference" "#PWR091"
 			(at 152.4 198.12 0)
 			(hide yes)
@@
 			(project "Poor86"
 				(path "/516eb290-d08d-4e43-95ba-5c21610df4ad/332916af-3e11-4b31-930a-ff884aaa5dd6"
-					(reference "#PWR095")
+					(reference "#PWR091")
 					(unit 1)
 				)
@@
 		(in_pos_files yes)
 		(dnp no)
-		(property "Reference" "U1"
+		(property "Reference" "U10"
 			(at 281.686 108.458 90)
 			(show_name no)
@@
 			(project "Poor86"
 				(path "/516eb290-d08d-4e43-95ba-5c21610df4ad/332916af-3e11-4b31-930a-ff884aaa5dd6"
-					(reference "U1")
+					(reference "U10")
 					(unit 8)
 				)
@@
 		(in_pos_files yes)
 		(dnp no)
-		(property "Reference" "R18"
+		(property "Reference" "R17"
 			(at 256.54 26.67 0)
 			(show_name no)
@@
 			(project "Poor86"
 				(path "/516eb290-d08d-4e43-95ba-5c21610df4ad/332916af-3e11-4b31-930a-ff884aaa5dd6"
-					(reference "R18")
+					(reference "R17")
 					(unit 1)
 				)
@@
 		(in_pos_files yes)
 		(dnp no)
-		(property "Reference" "JP3"
+		(property "Reference" "JP8"
 			(at 178.054 41.91 90)
 			(show_name no)
@@
 			(project "Poor86"
 				(path "/516eb290-d08d-4e43-95ba-5c21610df4ad/332916af-3e11-4b31-930a-ff884aaa5dd6"
-					(reference "JP3")
+					(reference "JP8")
 					(unit 1)
 				)
