File: PCB/external_perif.kicad_sch (KiCad schematic)
At the start: 15 parts, among them J1 Bus_ISA_8bit, J2 7-5530843-0, P1 USB_C_Plug_USB2.0, SW3 SW_Push_Dual, SW4 SW_Push_Dual, U11 CH552T, U5 ESP-12F

Commit message: more progress
Parts:
- removed J2: 7-5530843-0, ISA:TE_7-5530843-0, symbol isa:7-5530843-0
- added U7: RP2354B, Package_DFN_QFN:QFN-80-1EP_10x10mm_P0.4mm_EP3.4x3.4mm, symbol MCU_RaspberryPi:RP2354B
- D1: footprint Diode_SMD:D_0402_1005Metric -> Diode_SMD:D_1206_3216Metric_Pad1.42x1.75mm_HandSolder
- J1: footprint Connector_PinHeader_2.54mm:PinHeader_2x31_P2.54mm_Vertical_SMD -> ISA:TE_7-5530843-0
- P1: footprint Connector_USB:USB_C_Receptacle_GCT_USB4105-xx-A_16P_TopMnt_Horizontal -> (none)
- SW3, SW4: footprint Button_Switch_THT:SW_PUSH_6mm -> (none)
Connections:
- new net: U7.10 (DVDD), U7.32 (DVDD), U7.51 (DVDD)
- new net: U7.15 (IOVDD), U7.24 (IOVDD), U7.29 (IOVDD), U7.41 (IOVDD), U7.5 (IOVDD), U7.50 (IOVDD), U7.60 (IOVDD), U7.76 (IOVDD)
- new net A10: U7.8 (GPIO10)
- new net A11: U7.9 (GPIO11)
- new net A12: U7.11 (GPIO12)
- new net A13: U7.12 (GPIO13)
- new net A14: U7.13 (GPIO14)
- new net A15: U7.14 (GPIO15)
- new net A2: U7.79 (GPIO2)
- new net A3: U7.80 (GPIO3)
- new net A4: U7.1 (GPIO4)
- new net A5: U7.2 (GPIO5)
- new net A6: U7.3 (GPIO6)
- new net A7: U7.4 (GPIO7)
- new net A8: U7.6 (GPIO8)
- new net A9: U7.7 (GPIO9)
- new net D0: U7.16 (GPIO16)
- new net D1: U7.17 (GPIO17)
- new net D10: U7.27 (GPIO26)
- new net D11: U7.28 (GPIO27)
- new net D12: U7.36 (GPIO28)
- new net D13: U7.37 (GPIO29)
- new net D14: U7.38 (GPIO30)
- new net D15: U7.39 (GPIO31)
- new net D2: U7.18 (GPIO18)
- new net D3: U7.19 (GPIO19)
- new net D4: U7.20 (GPIO20)
- new net D5: U7.21 (GPIO21)
- new net D6: U7.22 (GPIO22)
- new net D7: U7.23 (GPIO23)
- new net D8: U7.25 (GPIO24)
- new net D9: U7.26 (GPIO25)
Other:
- moved on the sheet: J1, U5

Commit message: route-out in progress
Parts:
- added C35, C36, C45, C46, C47, C48, C49, C50: 2.2nF, Capacitor_SMD:C_01005_0402Metric, symbol Device:C_Small
- added J6: HDMI_A, Connector_Video:HDMI_A_Amphenol_10029449-x01xLF_Horizontal, symbol Connector:HDMI_A
- added U1: LFE5U-25F-6BG256C, ECP5:BGA256C80P16X16_1400X1400X170, symbol Lattice:LFE5U-25F-6BG256C
- J1: now not fitted; now left out of the parts list
- P1: footprint (none) -> Connector_USB:USB_C_Receptacle_GCT_USB4105-xx-A_16P_TopMnt_Horizontal
- SW3, SW4: footprint (none) -> Button_Switch_THT:SW_PUSH_6mm
- U7: private KLC_S4.2_VREG_LX -> (none); now not fitted; now left out of the parts list
Connections:
- net +3V3: now also U1.J6 (VCCIO6), U1.J7 (VCCIO6)
- net GNDD: now also J6.11 (CKS), J6.17 (GND), J6.2 (D2S), J6.5 (D1S), J6.8 (D0S), J6.SH
- new net: C35.2, J6.1 (D2+)
- new net: C49.2, J6.10 (CK+)
- new net: C50.2, J6.12 (CK-)
- new net: C36.2, J6.3 (D2-)
- new net: C45.2, J6.4 (D1+)
- new net: C46.2, J6.6 (D1-)
- new net: C47.2, J6.7 (D0+)
- new net: C48.2, J6.9 (D0-)
- new net CK+: C49.1, U1.L1 (PL26A)
- new net CK-: C50.1, U1.L2 (PL26B)
- new net D0+: C47.1, U1.M1 (PL26C)
- new net D0-: C48.1, U1.M2 (PL26D)
- new net D1+: C45.1, U1.N1 (PL32A)
- new net D1-: C46.1, U1.P2 (PL32B)
- new net D2+: C35.1, U1.P1 (PL35A)
- new net D2-: C36.1, U1.R1 (PL35B)

Commit message: Adding compact fpga on cpu pcb design
Parts:
- renumbered J1 to J2, R8 to R18, R9 to R19, R10 to R20, R11 to R21, R12 to R22, R13 to R23, U7 to U11
Connections:
- net D0: now also U1.P5 (PL47D)
- net D1: now also U1.N5 (PL44D)
- net D2: now also U1.P6 (PL47C)
- net D3: now also U1.N6 (PL47B)
- net Net-(J6-D2+): now reaches C35.2, J6.1 (D2+)
- net Net-(J6-CK+): now reaches C49.2, J6.10 (CK+)
- net Net-(J6-CK-): now reaches C50.2, J6.12 (CK-)
- net unconnected-(J6-CEC-Pad13): now reaches J6.13 (CEC)
- net unconnected-(J6-UTILITY-Pad14): now reaches J6.14 (UTILITY)
- net unconnected-(J6-SCL-Pad15): now reaches J6.15 (SCL)
- net unconnected-(J6-SDA-Pad16): now reaches J6.16 (SDA)
- net unconnected-(J6-+5V-Pad18): now reaches J6.18 (+5V)
- net unconnected-(J6-HPD-Pad19): now reaches J6.19 (HPD)
- net Net-(J6-D2-): now reaches C36.2, J6.3 (D2-)
- net Net-(J6-D1+): now reaches C45.2, J6.4 (D1+)
- net Net-(J6-D1-): now reaches C46.2, J6.6 (D1-)
- net Net-(J6-D0+): now reaches C47.2, J6.7 (D0+)
- net Net-(J6-D0-): now reaches C48.2, J6.9 (D0-)
- net Net-(U11-RST): now reaches C34.2, R18.1, SW3.1, SW3.3, U11.6 (RST)
- net Net-(R9-Pad1): now reaches R19.1, SW4.1, SW4.3
- net unconnected-(U5-~{RST}-Pad1): now reaches U5.1 (~{RST})
- net unconnected-(U5-MISO-Pad10): now reaches U5.10 (MISO)
- net unconnected-(U5-GPIO9-Pad11): now reaches U5.11 (GPIO9)
- net unconnected-(U5-GPIO10-Pad12): now reaches U5.12 (GPIO10)
- net unconnected-(U5-MOSI-Pad13): now reaches U5.13 (MOSI)
- net unconnected-(U5-SCLK-Pad14): now reaches U5.14 (SCLK)
- net unconnected-(U5-GND-Pad15): now reaches U5.15 (GND)
- net unconnected-(U5-GPIO15-Pad16): now reaches U5.16 (GPIO15)
- net unconnected-(U5-GPIO2-Pad17): now reaches U5.17 (GPIO2)
- net unconnected-(U5-GPIO0-Pad18): now reaches U5.18 (GPIO0)
- net unconnected-(U5-GPIO4-Pad19): now reaches U5.19 (GPIO4)
- net unconnected-(U5-ADC-Pad2): now reaches U5.2 (ADC)
- net unconnected-(U5-GPIO5-Pad20): now reaches U5.20 (GPIO5)
- net unconnected-(U5-GPIO3/RXD-Pad21): now reaches U5.21 (GPIO3/RXD)
- net unconnected-(U5-GPIO1/TXD-Pad22): now reaches U5.22 (GPIO1/TXD)
- net unconnected-(U5-EN-Pad3): now reaches U5.3 (EN)
- net unconnected-(U5-GPIO16-Pad4): now reaches U5.4 (GPIO16)
- net unconnected-(U5-GPIO14-Pad5): now reaches U5.5 (GPIO14)
- net unconnected-(U5-GPIO12-Pad6): now reaches U5.6 (GPIO12)
- net unconnected-(U5-GPIO13-Pad7): now reaches U5.7 (GPIO13)
- net unconnected-(U5-VCC-Pad8): now reaches U5.8 (VCC)
- net unconnected-(U5-CS0-Pad9): now reaches U5.9 (CS0)
- net Net-(U11-VBUS): now reaches P1.A4 (VBUS), P1.A9 (VBUS), P1.B4 (VBUS), P1.B9 (VBUS), U11.19 (VBUS)
- net unconnected-(U11-P32-Pad1): now reaches U11.1 (P32)
- net unconnected-(U11-P34-Pad12): now reaches U11.12 (P34)
- net unconnected-(U11-P35-Pad13): now reaches U11.13 (P35)
- net unconnected-(U11-P13-Pad16): now reaches U11.16 (P13)
- net unconnected-(U11-P12-Pad17): now reaches U11.17 (P12)
- net unconnected-(U11-P10-Pad7): now reaches U11.7 (P10)
- net unconnected-(U11-P11-Pad8): now reaches U11.8 (P11)
- net A21: now reaches U1.K4 (PL29A)
- net A20: now reaches U1.K5 (PL29B)
- net A20: now also U1.M5 (PL44C)
- net unconnected-(U1E-PL32C-PadL3): now reaches U1.L3 (PL32C)
- net A22: now reaches U1.L4 (PL29C)
- net A17: now reaches U1.L5 (PL29D)
- net A23: now reaches U1.M3 (PL32D)
- net A24: now reaches U1.M4 (PL35C)
- net A18: now reaches U1.M6 (PL47A)
- net A29: now reaches U1.N3 (PL35D)
- net A31: now reaches U1.N4 (PL38A)
- net A28: now reaches U1.P3 (PL38B)
- net A30: now reaches U1.P4 (PL41A)
- net A25: now reaches U1.R2 (PL38C)
- net A27: now reaches U1.R3 (PL41B)
- net unconnected-(U1E-PL41C-PadR4): now reaches U1.R4 (PL41C)
- net unconnected-(U1E-PL44A-PadR5): now reaches U1.R5 (PL44A)
- net A26: now reaches U1.T2 (PL38D)
- net unconnected-(U1E-PL41D-PadT3): now reaches U1.T3 (PL41D)
- net unconnected-(U1E-PL44B-PadT4): now reaches U1.T4 (PL44B)
