File: PCB/untitled.kicad_sch (KiCad schematic)
At the start: 3 parts, among them J2 5145154-4, J4 Bus_PCI_Express_x8, J5 10018783-10202TLF

Commit message: Adding compact fpga on cpu pcb design
Parts:
- renumbered J2 to J4, J4 to J5
Connections:
- net unconnected-(J5-PadA1): now reaches J5.A1
- net unconnected-(J5-PadA10): now reaches J5.A10
- net unconnected-(J5-PadA11): now reaches J5.A11
- net unconnected-(J5-PadA12): now reaches J5.A12
- net unconnected-(J5-PadA13): now reaches J5.A13
- net unconnected-(J5-PadA14): now reaches J5.A14
- net unconnected-(J5-PadA15): now reaches J5.A15
- net unconnected-(J5-PadA16): now reaches J5.A16
- net unconnected-(J5-PadA17): now reaches J5.A17
- net unconnected-(J5-PadA18): now reaches J5.A18
- net unconnected-(J5-PadA19): now reaches J5.A19
- net unconnected-(J5-PadA2): now reaches J5.A2
- net unconnected-(J5-PadA20): now reaches J5.A20
- net unconnected-(J5-PadA21): now reaches J5.A21
- net unconnected-(J5-PadA22): now reaches J5.A22
- net unconnected-(J5-PadA23): now reaches J5.A23
- net unconnected-(J5-PadA24): now reaches J5.A24
- net unconnected-(J5-PadA25): now reaches J5.A25
- net unconnected-(J5-PadA26): now reaches J5.A26
- net unconnected-(J5-PadA27): now reaches J5.A27
- net unconnected-(J5-PadA28): now reaches J5.A28
- net unconnected-(J5-PadA29): now reaches J5.A29
- net unconnected-(J5-PadA3): now reaches J5.A3
- net unconnected-(J5-PadA30): now reaches J5.A30
- net unconnected-(J5-PadA31): now reaches J5.A31
- net unconnected-(J5-PadA32): now reaches J5.A32
- net unconnected-(J5-PadA33): now reaches J5.A33
- net unconnected-(J5-PadA34): now reaches J5.A34
- net unconnected-(J5-PadA35): now reaches J5.A35
- net unconnected-(J5-PadA36): now reaches J5.A36
- net unconnected-(J5-PadA37): now reaches J5.A37
- net unconnected-(J5-PadA38): now reaches J5.A38
- net unconnected-(J5-PadA39): now reaches J5.A39
- net unconnected-(J5-PadA4): now reaches J5.A4
- net unconnected-(J5-PadA40): now reaches J5.A40
- net unconnected-(J5-PadA41): now reaches J5.A41
- net unconnected-(J5-PadA42): now reaches J5.A42
- net unconnected-(J5-PadA43): now reaches J5.A43
- net unconnected-(J5-PadA44): now reaches J5.A44
- net unconnected-(J5-PadA45): now reaches J5.A45
- net unconnected-(J5-PadA46): now reaches J5.A46
- net unconnected-(J5-PadA47): now reaches J5.A47
- net unconnected-(J5-PadA48): now reaches J5.A48
- net unconnected-(J5-PadA49): now reaches J5.A49
- net unconnected-(J5-PadA5): now reaches J5.A5
- net unconnected-(J5-PadA6): now reaches J5.A6
- net unconnected-(J5-PadA7): now reaches J5.A7
- net unconnected-(J5-PadA8): now reaches J5.A8
- net unconnected-(J5-PadA9): now reaches J5.A9
- net unconnected-(J5-PadB1): now reaches J5.B1
- net unconnected-(J5-PadB10): now reaches J5.B10
- net unconnected-(J5-PadB11): now reaches J5.B11
- net unconnected-(J5-PadB12): now reaches J5.B12
- net unconnected-(J5-PadB13): now reaches J5.B13
- net unconnected-(J5-PadB14): now reaches J5.B14
- net unconnected-(J5-PadB15): now reaches J5.B15
- net unconnected-(J5-PadB16): now reaches J5.B16
- net unconnected-(J5-PadB17): now reaches J5.B17
- net unconnected-(J5-PadB18): now reaches J5.B18
- net unconnected-(J5-PadB19): now reaches J5.B19
- net unconnected-(J5-PadB2): now reaches J5.B2
- net unconnected-(J5-PadB20): now reaches J5.B20
- net unconnected-(J5-PadB21): now reaches J5.B21
- net unconnected-(J5-PadB22): now reaches J5.B22
- net unconnected-(J5-PadB23): now reaches J5.B23
- net unconnected-(J5-PadB24): now reaches J5.B24
- net unconnected-(J5-PadB25): now reaches J5.B25
- net unconnected-(J5-PadB26): now reaches J5.B26
- net unconnected-(J5-PadB27): now reaches J5.B27
- net unconnected-(J5-PadB28): now reaches J5.B28
- net unconnected-(J5-PadB29): now reaches J5.B29
- net unconnected-(J5-PadB3): now reaches J5.B3
- net unconnected-(J5-PadB30): now reaches J5.B30
- net unconnected-(J5-PadB31): now reaches J5.B31
- net unconnected-(J5-PadB32): now reaches J5.B32
- net unconnected-(J5-PadB33): now reaches J5.B33
- net unconnected-(J5-PadB34): now reaches J5.B34
- net unconnected-(J5-PadB35): now reaches J5.B35
- net unconnected-(J5-PadB36): now reaches J5.B36
- net unconnected-(J5-PadB37): now reaches J5.B37
- net unconnected-(J5-PadB38): now reaches J5.B38
- net unconnected-(J5-PadB39): now reaches J5.B39
- net unconnected-(J5-PadB4): now reaches J5.B4
- net unconnected-(J5-PadB40): now reaches J5.B40
- net unconnected-(J5-PadB41): now reaches J5.B41
- net unconnected-(J5-PadB42): now reaches J5.B42
- net unconnected-(J5-PadB43): now reaches J5.B43
- net unconnected-(J5-PadB44): now reaches J5.B44
- net unconnected-(J5-PadB45): now reaches J5.B45
- net unconnected-(J5-PadB46): now reaches J5.B46
- net unconnected-(J5-PadB47): now reaches J5.B47
- net unconnected-(J5-PadB48): now reaches J5.B48
- net unconnected-(J5-PadB49): now reaches J5.B49
- net unconnected-(J5-PadB5): now reaches J5.B5
- net unconnected-(J5-PadB6): now reaches J5.B6
- net unconnected-(J5-PadB7): now reaches J5.B7
- net unconnected-(J5-PadB8): now reaches J5.B8
- net unconnected-(J5-PadB9): now reaches J5.B9
