File: PCB/video.kicad_sch (KiCad schematic)
At the start: 13 parts, among them U14 KM416x254, U15 KM416x254, U16 SN74ALVC164245DGG, U17 SN74ALVC164245DGG, U8 CL-GD5428-LOCALBUS

Commit message: More layout work
Connections:
- net +5V: now also U16.31 (V_{CC(A)}), U16.42 (V_{CC(A)}), U17.31 (V_{CC(A)}), U17.42 (V_{CC(A)})
- net 1A0: now also U8.54 (D0)
- net 1A1: now also U8.55 (D1)
- net 1A2: now also U8.56 (D2)
- net 1A3: now also U8.57 (D3)
- net 1A4: now also U8.59 (D4)
- net 1A5: now also U8.60 (D5)
- net 1A6: now also U8.62 (D6)
- net 1A7: now also U8.63 (D7)
- net 2A0: now also U8.11 (D8)
- net 2A1: now also U8.10 (D9)
- net 2A2: now also U8.9 (D10)
- net 2A3: now also U8.8 (D11)
- net 2A4: now also U8.6 (D12)
- net 2A5: now also U8.5 (D13)
- net 2A6: now also U8.4 (D14)
- net 2A7: now also U8.3 (D15)
- net D0: now also U16.2 (1B0); no longer U8.54 (D0)
- net D1: now also U16.3 (1B1); no longer U8.55 (D1)
- net D10: now also U16.16 (2B2); no longer U8.9 (D10)
- net D11: now also U16.17 (2B3); no longer U8.8 (D11)
- net D12: now also U16.19 (2B4); no longer U8.6 (D12)
- net D13: now also U16.20 (2B5); no longer U8.5 (D13)
- net D14: now also U16.22 (2B6); no longer U8.4 (D14)
- net D15: now also U16.23 (2B7); no longer U8.3 (D15)
- net D2: now also U16.5 (1B2); no longer U8.56 (D2)
- net D3: now also U16.6 (1B3); no longer U8.57 (D3)
- net D4: now also U16.8 (1B4); no longer U8.59 (D4)
- net D5: now also U16.9 (1B5); no longer U8.60 (D5)
- net D6: now also U16.11 (1B6); no longer U8.62 (D6)
- net D7: now also U16.12 (1B7); no longer U8.63 (D7)
- net D8: now also U16.13 (2B0); no longer U8.11 (D8)
- net D9: now also U16.14 (2B1); no longer U8.10 (D9)
- net GNDD: now also U16.10 (GND), U16.15 (GND), U16.21 (GND), U16.28 (GND), U16.34 (GND), U16.39 (GND), U16.4 (GND), U16.45 (GND), U17.10 (GND), U17.15 (GND), U17.21 (GND), U17.28 (GND), U17.34 (GND), U17.39 (GND), U17.4 (GND), U17.45 (GND)
- net W~{R}: now also U16.1 (1DIR), U16.24 (2DIR), U17.1 (1DIR), U17.24 (2DIR)
- net RESET: now reaches U8.46 (CPU_RESET)
- net D22: now reaches U17.11 (1B6)
- net D23: now reaches U17.12 (1B7)
- net D24: now reaches U17.13 (2B0)
- net D25: now reaches U17.14 (2B1)
- net D26: now reaches U17.16 (2B2)
- net D27: now reaches U17.17 (2B3)
- net D28: now reaches U17.19 (2B4)
- net D16: now reaches U17.2 (1B0)
- net D29: now reaches U17.20 (2B5)
- net D30: now reaches U17.22 (2B6)
- net D31: now reaches U17.23 (2B7)
- net D17: now reaches U17.3 (1B1)
- net D18: now reaches U17.5 (1B2)
- net D19: now reaches U17.6 (1B3)
- net D20: now reaches U17.8 (1B4)
- net D21: now reaches U17.9 (1B5)
- net CLK_CPU renamed CLK
- net ~{ADS_CPU} renamed ~{RDY}
- net ~{LBA_VGA}: no longer names the net of U8.22 (~{LBA})
- net ~{RDY_CPU} renamed ~{ADS}
- net ~{UADDR_VGA}: no longer names the net of U8.13 (NC/~{UADDR})
Other:
- note added: "When Direction is low, the data points to the A side. B -> A (Read, the CL-GD54xx drives the bus). The CL-GD54xx decides when to assert the OE"
- moved on the sheet: U16, U17

Commit message: route-out in progress
Parts:
- C37, C38, C39, C40, C41, C42, C43, C44, U14, U15, U16, U17, U8: now not fitted; now left out of the parts list

Commit message: Adding compact fpga on cpu pcb design
Parts:
- renumbered C41 to C43, C40 to C44, C42 to C45, C39 to C46, C43 to C47, C38 to C48, C44 to C49, C37 to C50, U16 to U14, U17 to U15, U8 to U16, U14 to U17, U15 to U18
Changed lines of the file:
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@@
 		(dnp yes)
 		(fields_autoplaced yes)
-		(property "Reference" "#PWR076"
+		(property "Reference" "#PWR0103"
 			(at -34.29 186.69 0)
 			(hide yes)
@@
 			(project "Poor86"
 				(path "/516eb290-d08d-4e43-95ba-5c21610df4ad/8f55fba7-2b48-44e0-a4b2-bfc9178c5413"
-					(reference "#PWR076")
+					(reference "#PWR0103")
 					(unit 1)
 				)
@@
 		(in_pos_files yes)
 		(dnp yes)
-		(property "Reference" "C38"
+		(property "Reference" "C48"
 			(at 214.63 110.49 0)
 			(show_name no)
@@
 			(project "Poor86"
 				(path "/516eb290-d08d-4e43-95ba-5c21610df4ad/8f55fba7-2b48-44e0-a4b2-bfc9178c5413"
-					(reference "C38")
+					(reference "C48")
 					(unit 1)
 				)
@@
 		(in_pos_files yes)
 		(dnp yes)
-		(property "Reference" "C43"
+		(property "Reference" "C47"
 			(at 214.63 60.96 0)
 			(show_name no)
@@
 			(project "Poor86"
 				(path "/516eb290-d08d-4e43-95ba-5c21610df4ad/8f55fba7-2b48-44e0-a4b2-bfc9178c5413"
-					(reference "C43")
+					(reference "C47")
 					(unit 1)
 				)
@@
 		(dnp no)
 		(fields_autoplaced yes)
-		(property "Reference" "#PWR072"
+		(property "Reference" "#PWR0108"
 			(at 82.55 198.12 0)
 			(hide yes)
@@
 			(project "Poor86"
 				(path "/516eb290-d08d-4e43-95ba-5c21610df4ad/8f55fba7-2b48-44e0-a4b2-bfc9178c5413"
-					(reference "#PWR072")
+					(reference "#PWR0108")
 					(unit 1)
 				)
@@
 		(dnp yes)
 		(fields_autoplaced yes)
-		(property "Reference" "#PWR084"
+		(property "Reference" "#PWR0111"
 			(at 223.52 63.5 0)
 			(hide yes)
@@
 			(project "Poor86"
 				(path "/516eb290-d08d-4e43-95ba-5c21610df4ad/8f55fba7-2b48-44e0-a4b2-bfc9178c5413"
-					(reference "#PWR084")
+					(reference "#PWR0111")
 					(unit 1)
 				)
@@
 		(in_pos_files yes)
 		(dnp yes)
-		(property "Reference" "C37"
+		(property "Reference" "C50"
 			(at 219.71 110.49 0)
 			(show_name no)
@@
 			(project "Poor86"
 				(path "/516eb290-d08d-4e43-95ba-5c21610df4ad/8f55fba7-2b48-44e0-a4b2-bfc9178c5413"
-					(reference "C37")
+					(reference "C50")
 					(unit 1)
 				)
@@
 		(in_pos_files no)
 		(dnp yes)
-		(property "Reference" "#PWR086"
+		(property "Reference" "#PWR0105"
 			(at -31.75 123.19 0)
 			(hide yes)
@@
 			(project "Poor86"
 				(path "/516eb290-d08d-4e43-95ba-5c21610df4ad/8f55fba7-2b48-44e0-a4b2-bfc9178c5413"
-					(reference "#PWR086")
+					(reference "#PWR0105")
 					(unit 1)
 				)
@@
 		(dnp yes)
 		(fields_autoplaced yes)
-		(property "Reference" "U15"
+		(property "Reference" "U18"
 			(at 234.95 68.58 0)
 			(show_name no)
@@
 			(project "Poor86"
 				(path "/516eb290-d08d-4e43-95ba-5c21610df4ad/8f55fba7-2b48-44e0-a4b2-bfc9178c5413"
-					(reference "U15")
+					(reference "U18")
 					(unit 1)
 				)
@@
 		(in_pos_files yes)
 		(dnp yes)
-		(property "Reference" "C41"
+		(property "Reference" "C43"
 			(at 205.74 60.96 0)
 			(show_name no)
@@
 			(project "Poor86"
 				(path "/516eb290-d08d-4e43-95ba-5c21610df4ad/8f55fba7-2b48-44e0-a4b2-bfc9178c5413"
-					(reference "C41")
+					(reference "C43")
 					(unit 1)
 				)
@@
 		(dnp yes)
 		(fields_autoplaced yes)
-		(property "Reference" "#PWR075"
+		(property "Reference" "#PWR0110"
 			(at 201.93 118.11 0)
 			(hide yes)
@@
 			(project "Poor86"
 				(path "/516eb290-d08d-4e43-95ba-5c21610df4ad/8f55fba7-2b48-44e0-a4b2-bfc9178c5413"
-					(reference "#PWR075")
+					(reference "#PWR0110")
 					(unit 1)
 				)
@@
 		(dnp yes)
 		(fields_autoplaced yes)
-		(property "Reference" "#PWR082"
+		(property "Reference" "#PWR0112"
 			(at 223.52 113.03 0)
 			(hide yes)
@@
 			(project "Poor86"
 				(path "/516eb290-d08d-4e43-95ba-5c21610df4ad/8f55fba7-2b48-44e0-a4b2-bfc9178c5413"
-					(reference "#PWR082")
+					(reference "#PWR0112")
 					(unit 1)
 				)
@@
 		(dnp yes)
 		(fields_autoplaced yes)
-		(property "Reference" "#PWR074"
+		(property "Reference" "#PWR0102"
 			(at -35.56 106.68 0)
 			(hide yes)
@@
 			(project "Poor86"
 				(path "/516eb290-d08d-4e43-95ba-5c21610df4ad/8f55fba7-2b48-44e0-a4b2-bfc9178c5413"
-					(reference "#PWR074")
+					(reference "#PWR0102")
 					(unit 1)
 				)
@@
 		(dnp no)
 		(fields_autoplaced yes)
-		(property "Reference" "#PWR077"
+		(property "Reference" "#PWR0107"
 			(at 62.23 187.96 0)
 			(hide yes)
@@
 			(project "Poor86"
 				(path "/516eb290-d08d-4e43-95ba-5c21610df4ad/8f55fba7-2b48-44e0-a4b2-bfc9178c5413"
-					(reference "#PWR077")
+					(reference "#PWR0107")
 					(unit 1)
 				)
@@
 		(in_pos_files yes)
 		(dnp yes)
-		(property "Reference" "C42"
+		(property "Reference" "C45"
 			(at 210.82 60.96 0)
 			(show_name no)
@@
 			(project "Poor86"
 				(path "/516eb290-d08d-4e43-95ba-5c21610df4ad/8f55fba7-2b48-44e0-a4b2-bfc9178c5413"
-					(reference "C42")
+					(reference "C45")
 					(unit 1)
 				)
@@
 		(dnp yes)
 		(fields_autoplaced yes)
-		(property "Reference" "#PWR083"
+		(property "Reference" "#PWR0109"
 			(at 201.93 68.58 0)
 			(hide yes)
@@
 			(project "Poor86"
 				(path "/516eb290-d08d-4e43-95ba-5c21610df4ad/8f55fba7-2b48-44e0-a4b2-bfc9178c5413"
-					(reference "#PWR083")
+					(reference "#PWR0109")
 					(unit 1)
 				)
@@
 		(dnp yes)
 		(fields_autoplaced yes)
-		(property "Reference" "#PWR085"
+		(property "Reference" "#PWR0104"
 			(at -33.02 43.18 0)
 			(hide yes)
@@
 			(project "Poor86"
 				(path "/516eb290-d08d-4e43-95ba-5c21610df4ad/8f55fba7-2b48-44e0-a4b2-bfc9178c5413"
-					(reference "#PWR085")
+					(reference "#PWR0104")
 					(unit 1)
 				)
@@
 		(in_pos_files yes)
 		(dnp yes)
-		(property "Reference" "C39"
+		(property "Reference" "C46"
 			(at 210.82 110.49 0)
 			(show_name no)
@@
 			(project "Poor86"
 				(path "/516eb290-d08d-4e43-95ba-5c21610df4ad/8f55fba7-2b48-44e0-a4b2-bfc9178c5413"
-					(reference "C39")
+					(reference "C46")
 					(unit 1)
 				)
@@
 		(dnp yes)
 		(fields_autoplaced yes)
-		(property "Reference" "U14"
+		(property "Reference" "U17"
 			(at 234.95 19.05 0)
 			(show_name no)
@@
 			(project "Poor86"
 				(path "/516eb290-d08d-4e43-95ba-5c21610df4ad/8f55fba7-2b48-44e0-a4b2-bfc9178c5413"
-					(reference "U14")
+					(reference "U17")
 					(unit 1)
 				)
@@
 		(dnp yes)
 		(fields_autoplaced yes)
-		(property "Reference" "U8"
+		(property "Reference" "U16"
 			(at 138.0333 19.685 0)
 			(show_name no)
@@
 			(project "Poor86"
 				(path "/516eb290-d08d-4e43-95ba-5c21610df4ad/8f55fba7-2b48-44e0-a4b2-bfc9178c5413"
-					(reference "U8")
+					(reference "U16")
 					(unit 1)
 				)
@@
 		(in_pos_files yes)
 		(dnp yes)
-		(property "Reference" "C44"
+		(property "Reference" "C49"
 			(at 219.71 60.96 0)
 			(show_name no)
@@
 			(project "Poor86"
 				(path "/516eb290-d08d-4e43-95ba-5c21610df4ad/8f55fba7-2b48-44e0-a4b2-bfc9178c5413"
-					(reference "C44")
+					(reference "C49")
 					(unit 1)
 				)
@@
 		(dnp yes)
 		(fields_autoplaced yes)
-		(property "Reference" "U16"
+		(property "Reference" "U14"
 			(at -33.4167 100.33 0)
 			(show_name no)
@@
 			(project "Poor86"
 				(path "/516eb290-d08d-4e43-95ba-5c21610df4ad/8f55fba7-2b48-44e0-a4b2-bfc9178c5413"
-					(reference "U16")
+					(reference "U14")
 					(unit 1)
 				)
@@
 		(dnp yes)
 		(fields_autoplaced yes)
-		(property "Reference" "U17"
+		(property "Reference" "U15"
 			(at -32.1467 180.34 0)
 			(show_name no)
@@
 			(project "Poor86"
 				(path "/516eb290-d08d-4e43-95ba-5c21610df4ad/8f55fba7-2b48-44e0-a4b2-bfc9178c5413"
-					(reference "U17")
+					(reference "U15")
 					(unit 1)
 				)
@@
 		(in_pos_files yes)
 		(dnp yes)
-		(property "Reference" "C40"
+		(property "Reference" "C44"
 			(at 205.74 110.49 0)
 			(show_name no)
@@
 			(project "Poor86"
 				(path "/516eb290-d08d-4e43-95ba-5c21610df4ad/8f55fba7-2b48-44e0-a4b2-bfc9178c5413"
-					(reference "C40")
+					(reference "C44")
 					(unit 1)
 				)
@@
 		(dnp no)
 		(fields_autoplaced yes)
-		(property "Reference" "#PWR073"
+		(property "Reference" "#PWR0106"
 			(at 17.78 81.28 0)
 			(hide yes)
@@
 			(project "Poor86"
 				(path "/516eb290-d08d-4e43-95ba-5c21610df4ad/8f55fba7-2b48-44e0-a4b2-bfc9178c5413"
-					(reference "#PWR073")
+					(reference "#PWR0106")
 					(unit 1)
 				)
